File: duplicate_sensors.kicad_sch (KiCad schematic)
At the start: 12 parts, among them J1 AOM-5035L-HD3-LW100, Q1 AO3400A

Commit message: adding footprints to sensors
Parts:
- removed C2: 1e-6, symbol Device:C
- removed R5, R7: 100k, Package_TO_SOT_SMD:SOT-23-5, symbol Device:R
- removed R6: 100K, Package_TO_SOT_SMD:SOT-23-5, symbol Device:R
- C42: renamed from C1; value 1e-6F -> 10nF
- R56: renamed from R1; value 5.6k -> 1k
- renumbered J1 to J16, Q1 to Q2, R3 to R57, R4 to R58, R2 to R59, TSAL6200 to TSAL1
Connections:
- net +3.3V: now also J16.2 (Pin_2); no longer C42.1, J16.1 (Pin_1)
- net GND: now also C42.2; no longer R56.1
- net at R56.2: now also C42.1; no longer J16.2 (Pin_2)
- new net: J16.1 (Pin_1), R56.1
Other:
- moved on the sheet: C42, Q2, R56, R57, R58, R59, TSAL1

Commit message: Revert "Merge branch 'main' of https://github.com/pequeno212/PCB_SeniorDesign_team20"
This reverts commit 8ddd870afa6ea88a1f78691f7845b0b29e49b9ae, reversing
changes made to b7b9844e80cb26773f88e7278ccd95378529a98d.
Parts:
- removed C42: 10nF, symbol Device:C
- removed J16: AOM-5035L-HD3-LW100, Connector_Audio:Jack_XLR_Neutrik_NC3FAAH_Horizontal, symbol Connector_Generic:Conn_01x03
- removed R56: 1k, symbol Device:R
- added C1: 1e-7, symbol Device:C
- added J1: MIC_I2S_CONNECTOR, symbol Connector_Generic:Conn_01x06
- R3: renamed from R57; value 100 -> 10
- renumbered Q2 to Q1, R59 to R2, R58 to R4, TSAL1 to TSAL6200
Connections:
- net GND: now also C1.2, J1.1 (Pin_1), J1.5 (Pin_5)
- net +3.3V renamed +3V3
- net +3V3: now also C1.1, J1.6 (Pin_6)
Other:
- note added: "J1 - 6 Pin Connector to Adafruit ICS-43434 Breakout 1 - SEL → GND 2 - LRCL → MIC_I2S_WS 3 - DOUT → MIC_I2S_SD 4 - BCLK → MIC_I2S_SCK 5 - GND → GND 6 - 3V → +3V3"
- note added: "https://www.digikey.com/en/products/detail/vishay-semiconductor-opto-division/TSAL6200/1681339"
- moved on the sheet: Q1, R2, R3, R4, TSAL6200
