File: duplicate_sensors.kicad_sch (KiCad schematic)
At the start: 12 parts, among them J1 AOM-5035L-HD3-LW100, Q1 AO3400A

Commit message: Finished Digital MIC + IR
Parts:
- removed C2: 1e-6, symbol Device:C
- removed J1: AOM-5035L-HD3-LW100, Connector_Audio:Jack_XLR_Neutrik_NC3FAAH_Horizontal, symbol Connector_Generic:Conn_01x03
- removed R1: 5.6k, symbol Device:R
- removed R5, R7: 100k, Package_TO_SOT_SMD:SOT-23-5, symbol Device:R
- removed R6: 100K, Package_TO_SOT_SMD:SOT-23-5, symbol Device:R
- added J1: MIC_I2S_CONNECTOR, symbol Connector_Generic:Conn_01x06
- C1: value 1e-6F -> 1e-7
- R3: value 100 -> 10
Connections:
- net GND: now also C1.2, J1.1 (Pin_1), J1.5 (Pin_5)
- net +3.3V renamed +3V3
- net +3V3: now also J1.6 (Pin_6)
Other:
- note added: "J1 - 6 Pin Connector to Adafruit ICS-43434 Breakout 1 - SEL → GND 2 - LRCL → MIC_I2S_WS 3 - DOUT → MIC_I2S_SD 4 - BCLK → MIC_I2S_SCK 5 - GND → GND 6 - 3V → +3V3"
- note added: "https://www.digikey.com/en/products/detail/vishay-semiconductor-opto-division/TSAL6200/1681339"

Commit message: Major Changes - Schematic Done??
Parts:
- removed C1: 1e-7, symbol Device:C
- removed J1: MIC_I2S_CONNECTOR, symbol Connector_Generic:Conn_01x06
- added C44: 100n, Capacitor_SMD:C_0603_1608Metric, symbol Device:C
- added J19: MIC_I2S_CONNECTOR, Connector_PinSocket_2.54mm:PinSocket_1x06_P2.54mm_Vertical, symbol Connector_Generic:Conn_01x06
- R65: renamed from R3; footprint Package_DIP:DIP-8_W7.62mm -> Resistor_SMD:R_0603_1608Metric
- R66: renamed from R4; value 100k -> 10k; footprint Package_DIP:DIP-8_W7.62mm -> Resistor_SMD:R_0603_1608Metric
- R67: renamed from R2; value 39 -> 17; footprint Package_DIP:DIP-8_W7.62mm -> Resistor_SMD:R_0603_1608Metric
- TSAL1: renamed from TSAL6200; footprint Package_DirectFET:DirectFET_MD -> LED_SMD:LED_0603_1608Metric
- renumbered Q1 to Q3
Connections:
- net GND: now also C44.2, J19.1 (Pin_1), J19.5 (Pin_5)
- net TV_IR_PWM: now also R65.2
- net +3V3 renamed 3V3
- net 3V3: now also C44.1, J19.6 (Pin_6)
- new net I2S3_CK: J19.4 (Pin_4)
- new net I2S3_SD: J19.3 (Pin_3)
- new net I2S3_WS: J19.2 (Pin_2)
Other:
- note added: "Digital microphone website : https://www.adafruit.com/product/6049"
- note added: "IR EMITTER"
- moved on the sheet: Q3, R65, R66, R67, TSAL1
