File: Analog.kicad_sch (KiCad schematic)
At the start: 25 parts, among them J2 Conn_01x02_Socket, J3 Conn_01x02_Socket, J9 Conn_01x02_Socket, U10 MAX98357A, U3 MAX98357A, U7 TLV172IDCK, U8 TPS60400DBV, U9 TLV172IDCK

Commit message: STM32 Work
Connections:
- net SD_MODE renamed DAC_LEFT_SD_MODE
- net DAC_LEFT_SD_MODE: no longer R32.1
- new net DAC_RIGHT_SD_MODE: R32.1
Other:
- note added: "LEFT CHANNEL"
- note added: "RIGHT CHANNEL"
Changed lines of the file:
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@@
 		)
 	)
+	(text "LEFT CHANNEL"
+		(exclude_from_sim no)
+		(at 108.712 36.576 0)
+		(effects
+			(font
+				(size 2.54 2.54)
+			)
+		)
+	)
 	(text "sensitivity = -44dB ==> 10^(-44/20) = 6.31mVrms per pascal = +-89mV\ngain of 18 to get +- 1.6V\nadd 1.65V to get .05V to 3.25V swing\n\n\n"
 		(exclude_from_sim no)
@@
 		)
 	)
+	(text "RIGHT CHANNEL\n"
+		(exclude_from_sim no)
+		(at 194.056 37.846 0)
+		(effects
+			(font
+				(size 2.54 2.54)
+			)
+		)
+	)
+	(text_box "Gain: Connect to VDD = 6dB"
+		(exclude_from_sim no)
+		(at 60.96 67.31 0)
+		(size 19.05 5.9929)
+		(margins 0.9525 0.9525 0.9525 0.9525)
+		(stroke
+			(width 0)
+			(type solid)
+		)
+		(fill
+			(type none)
+		)
+		(effects
+			(font
+				(size 1.27 1.27)
+			)
+			(justify left top)
+		)
+	)
 	(junction
 		(at 77.47 123.19)
@@
 		)
 	)
-	(hierarchical_label "SD_MODE"
+	(hierarchical_label "DAC_LEFT_SD_MODE"
 		(shape input)
 		(at 55.88 55.88 180)
@@
 		)
 	)
+	(hierarchical_label "DAC_RIGHT_SD_MODE"
+		(shape input)
+		(at 185.42 55.88 180)
+		(effects
+			(font
+				(size 1.27 1.27)
+			)
+			(justify right)
+		)
+	)
 	(hierarchical_label "MIC"
 		(shape input)
@@
 		)
 	)
-	(hierarchical_label "SD_MODE"
-		(shape input)
-		(at 185.42 55.88 180)
-		(effects
-			(font
-				(size 1.27 1.27)
-			)
-			(justify right)
-		)
-	)
 	(symbol
 		(lib_id "power:GND")
@@
 		)
 		(property "Value" "-3V3"
-			(at 107.95 129.794 0)
+			(at 110.49 132.08 0)
 			(show_name no)
 			(do_not_autoplace no)

Commit message: monkey business
Parts:
- C34: footprint Package_TO_SOT_SMD:SOT-23-5 -> Capacitor_SMD:C_0603_1608Metric
- J2: footprint Package_SO:HTSSOP-20-1EP_4.4x6.5mm_P0.65mm_EP3.4x6.5mm_ThermalVias -> Connector_PinHeader_2.54mm:PinHeader_1x02_P2.54mm_Vertical
- gave numbers to parts that had none: 2
Changed lines of the file:
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@@
 			)
 		)
-		(property "Footprint" "Package_TO_SOT_SMD:SOT-23-5"
+		(property "Footprint" "Capacitor_SMD:C_0603_1608Metric"
 			(at 63.1952 185.42 0)
 			(hide yes)
@@
 		(dnp no)
 		(fields_autoplaced yes)
-		(property "Reference" "C?"
+		(property "Reference" "C37"
 			(at 48.26 67.3099 0)
 			(show_name no)
@@
 			(project "SeniorDesign_PCB"
 				(path "/88e1ced0-9576-4565-ab29-f74bf51ccbda/f9ef2c8a-940c-4bd3-9d49-5676059e2f63"
-					(reference "C?")
+					(reference "C37")
 					(unit 1)
 				)
@@
 		(dnp no)
 		(fields_autoplaced yes)
-		(property "Reference" "C?"
+		(property "Reference" "C38"
 			(at 34.29 67.3099 0)
 			(show_name no)
@@
 			(project "SeniorDesign_PCB"
 				(path "/88e1ced0-9576-4565-ab29-f74bf51ccbda/f9ef2c8a-940c-4bd3-9d49-5676059e2f63"
-					(reference "C?")
+					(reference "C38")
 					(unit 1)
 				)
@@
 			)
 		)
-		(property "Footprint" "Package_SO:HTSSOP-20-1EP_4.4x6.5mm_P0.65mm_EP3.4x6.5mm_ThermalVias"
+		(property "Footprint" "Connector_PinHeader_2.54mm:PinHeader_1x02_P2.54mm_Vertical"
 			(at 66.04 125.73 0)
 			(hide yes)
