File: Analog.kicad_sch (KiCad schematic)
At the start: 25 parts, among them J2 Conn_01x02_Socket, J3 Conn_01x02_Socket, J9 Conn_01x02_Socket, U10 MAX98357A, U3 MAX98357A, U7 TLV172IDCK, U8 TPS60400DBV, U9 TLV172IDCK

Commit message: Major Changes - Schematic Done??
Parts:
- removed C34: 1u, Capacitor_SMD:C_0603_1608Metric, symbol Device:C
- removed U8: TPS60400DBV, Package_TO_SOT_SMD:SOT-23-5, symbol Regulator_SwitchedCapacitor:TPS60400DBV
- added C40, C44: 100n, Capacitor_SMD:C_0603_1608Metric, symbol Device:C
- added R34, R35: 0R, Resistor_SMD:R_0603_1608Metric, symbol Device:R
- added U16: TLV172IDCK, Package_TO_SOT_SMD:SOT-353_SC-70-5, symbol Amplifier_Operational:TLV172IDCK
- C13: renamed from C37; value 0.1u -> 100n
- C17: renamed from C36; value 0.1u -> 100n
- J6: renamed from J2; footprint Connector_PinHeader_2.54mm:PinHeader_1x02_P2.54mm_Vertical -> Connector_PinSocket_2.54mm:PinSocket_1x02_P2.54mm_Vertical
- J7: renamed from J3; footprint (none) -> Connector_PinSocket_2.54mm:PinSocket_1x02_P2.54mm_Vertical
- J8: renamed from J9; footprint (none) -> Connector_PinSocket_2.54mm:PinSocket_1x02_P2.54mm_Vertical
- R20: renamed from R?; value 210k -> 0R
- R21: renamed from R5; value 2.2k -> 2k2
- R30: renamed from R32; value 0 -> 210k
- renumbered C38 to C12, C29 to C15, C35 to C16, R30 to R22, R31 to R23, R28 to R24, R29 to R25, R22 to R27, R25 to R28, R27 to R29, U3 to U5, U9 to U6, U10 to U8
Connections:
- net +3V3 is gone; now on net 3V3: C12.1, C13.1, C16.1, C17.1, R21.1, R24.2, U6.5 (V+), U7.5 (V+)
- net -3V3: now also U7.2 (V-), U16.2 (V-)
- net GND: now also C40.2, C44.2; no longer U7.2 (V-)
- net at R24.1, R25.2: now also U16.1 (+); no longer R26.1
- net +3V renamed 3V3
- net 3V3: now also C40.1, C44.1, R34.1, R35.1, U16.5 (V+); no longer U5.2 (GAIN_SLOT), U8.2 (GAIN_SLOT)
- net I2S3_CK renamed I2S2_CK
- net I2S3_SD renamed I2S2_SD
- net I2S3_WS renamed I2S2_WS
- net SD_MODE renamed LEFT_SD_MODE
- net LEFT_SD_MODE: no longer R30.1
- new net: R34.2, U8.2 (GAIN_SLOT)
- new net: R26.1, U16.3 (-), U16.4
- new net: R35.2, U5.2 (GAIN_SLOT)
- new net RIGHT_SD_MODE: R30.1
Other:
- note added: "LEFT SPEAKER"
- note added: "RIGHT SPEAKER"
- note removed: "Charge Pump: -3V3"
- moved on the sheet: C12, C13, C15, C16, C17, J6, R21, R22, R23, R24, R25, R27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

Commit message: Almost Done with Dev Board
Parts:
- added C53: 100n, Capacitor_SMD:C_0603_1608Metric, symbol Device:C
Connections:
- net 3V3: now also C53.1
- net GND: now also C53.2

Commit message: Minor PCB Changes
Parts:
- J6, J7, J8: footprint Connector_PinSocket_2.54mm:PinSocket_1x02_P2.54mm_Vertical -> Connector_PinHeader_2.54mm:PinHeader_1x02_P2.54mm_Vertical
Changed lines of the file:
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@@
 			)
 		)
-		(property "Footprint" "Connector_PinSocket_2.54mm:PinSocket_1x02_P2.54mm_Vertical"
+		(property "Footprint" "Connector_PinHeader_2.54mm:PinHeader_1x02_P2.54mm_Vertical"
 			(at 66.04 133.35 0)
 			(hide yes)
@@
 			)
 		)
-		(property "Footprint" "Connector_PinSocket_2.54mm:PinSocket_1x02_P2.54mm_Vertical"
+		(property "Footprint" "Connector_PinHeader_2.54mm:PinHeader_1x02_P2.54mm_Vertical"
 			(at 241.3 45.72 0)
 			(hide yes)
@@
 			)
 		)
-		(property "Footprint" "Connector_PinSocket_2.54mm:PinSocket_1x02_P2.54mm_Vertical"
+		(property "Footprint" "Connector_PinHeader_2.54mm:PinHeader_1x02_P2.54mm_Vertical"
 			(at 111.76 45.72 0)
 			(hide yes)
