File: SeniorDesign_PCB.kicad_pcb (KiCad board)
At the start: 0 parts

Commit message: Major Changes - Schematic Done??
Other:
- copper layers 0 -> 2
Changed lines of the file:
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@@
-(kicad_pcb (version 20260206) (generator "pcbnew") (generator_version "10.0")
+(kicad_pcb
+	(version 20260206)
+	(generator "pcbnew")
+	(generator_version "10.0")
+	(general
+		(thickness 1.6)
+		(legacy_teardrops no)
+	)
+	(paper "A4")
+	(layers
+		(0 "F.Cu" signal)
+		(2 "B.Cu" signal)
+		(9 "F.Adhes" user "F.Adhesive")
+		(11 "B.Adhes" user "B.Adhesive")
+		(13 "F.Paste" user)
+		(15 "B.Paste" user)
+		(5 "F.SilkS" user "F.Silkscreen")
+		(7 "B.SilkS" user "B.Silkscreen")
+		(1 "F.Mask" user)
+		(3 "B.Mask" user)
+		(17 "Dwgs.User" user "User.Drawings")
+		(19 "Cmts.User" user "User.Comments")
+		(21 "Eco1.User" user "User.Eco1")
+		(23 "Eco2.User" user "User.Eco2")
+		(25 "Edge.Cuts" user)
+		(27 "Margin" user)
+		(31 "F.CrtYd" user "F.Courtyard")
+		(29 "B.CrtYd" user "B.Courtyard")
+		(35 "F.Fab" user)
+		(33 "B.Fab" user)
+		(39 "User.1" user)
+		(41 "User.2" user)
+		(43 "User.3" user)
+		(45 "User.4" user)
+	)
+	(setup
+		(pad_to_mask_clearance 0)
+		(allow_soldermask_bridges_in_footprints no)
+		(tenting
+			(front yes)
+			(back yes)
+		)
+		(covering
+			(front no)
+			(back no)
+		)
+		(plugging
+			(front no)
+			(back no)
+		)
+		(capping no)
+		(filling no)
+		(pcbplotparams
+			(layerselection 0x00000000_00000000_55555555_5755f5ff)
+			(plot_on_all_layers_selection 0x00000000_00000000_00000000_00000000)
+			(disableapertmacros no)
+			(usegerberextensions no)
+			(usegerberattributes yes)
+			(usegerberadvancedattributes yes)
+			(creategerberjobfile yes)
+			(dashed_line_dash_ratio 12)
+			(dashed_line_gap_ratio 3)
+			(svgprecision 4)
+			(plotframeref no)
+			(mode 1)
+			(useauxorigin no)
+			(pdf_front_fp_property_popups yes)
+			(pdf_back_fp_property_popups yes)
+			(pdf_metadata yes)
+			(pdf_single_document no)
+			(dxfpolygonmode yes)
+			(dxfimperialunits yes)
+			(dxfusepcbnewfont yes)
+			(psnegative no)
+			(psa4output no)
+			(plot_black_and_white yes)
+			(sketchpadsonfab no)
+			(plotpadnumbers no)
+			(hidednponfab no)
+			(sketchdnponfab yes)
+			(crossoutdnponfab yes)
+			(subtractmaskfromsilk no)
+			(outputformat 1)
+			(mirror no)
+			(drillshape 1)
+			(scaleselection 1)
+			(outputdirectory "")
+		)
+	)
+	(embedded_fonts no)
 )

Commit message: PCB Start, Schematic polish
Parts:
- added AE1: Antenna, RF_Antenna:Texas_SWRA117D_2.4GHz_Left, F.Cu at (106.6, 184.4)
- added C1: 1u, Capacitor_SMD:C_0603_1608Metric, B.Cu at (103.2, 139.8)
- added C10: 100n, Capacitor_SMD:C_0603_1608Metric, B.Cu at (110.2, 131.1)
- added C11: 100n, Capacitor_SMD:C_0603_1608Metric, F.Cu at (121.7, 141.3)
- added C12: 10u, Capacitor_SMD:C_0603_1608Metric, F.Cu at (186.9, 82.5)
- added C13: 100n, Capacitor_SMD:C_0603_1608Metric, F.Cu at (186.9, 85.0)
- added C14: 100n, Capacitor_SMD:C_0603_1608Metric, F.Cu at (188.7, 133.3)
- added C15: 1uF, Capacitor_SMD:C_0603_1608Metric, F.Cu at (186.9, 87.5)
- added C16: 10u, Capacitor_SMD:C_0603_1608Metric, F.Cu at (186.9, 90.0)
- added C17: 100n, Capacitor_SMD:C_0603_1608Metric, F.Cu at (186.9, 92.6)
- added C18: 100n, Capacitor_SMD:C_0603_1608Metric, F.Cu at (196.3, 38.3)
- added C19: 100n, Capacitor_SMD:C_0603_1608Metric, F.Cu at (196.3, 40.8)
- added C2: 100n, Capacitor_SMD:C_0603_1608Metric, B.Cu at (107.4, 139.8)
- added C20: 4u7, Capacitor_SMD:C_0603_1608Metric, F.Cu at (196.3, 43.4)
- added C21: 22u, Capacitor_SMD:C_0603_1608Metric, F.Cu at (196.3, 45.9)
- added C22: 1u, Capacitor_SMD:C_0603_1608Metric, F.Cu at (80.6, 49.5)
- added C23: 1u, Capacitor_SMD:C_0603_1608Metric, F.Cu at (80.6, 52.0)
- added C24: 100n, Capacitor_SMD:C_0603_1608Metric, F.Cu at (80.6, 54.5)
- added C25: 100n, Capacitor_SMD:C_0603_1608Metric, F.Cu at (80.6, 57.1)
- added C26: 22p, Capacitor_SMD:C_0603_1608Metric, F.Cu at (83.7, 162.4)
- added C27: 22p, Capacitor_SMD:C_0603_1608Metric, F.Cu at (83.7, 164.9)
- added C28: DNP, Capacitor_SMD:C_0402_1005Metric, F.Cu at (105.7, 162.2)
- added C29: DNP, Capacitor_SMD:C_0402_1005Metric, F.Cu at (105.7, 164.1)
- added C3: 100n, Capacitor_SMD:C_0603_1608Metric, B.Cu at (105.4, 139.8)
- added C30: DNP, Capacitor_SMD:C_0402_1005Metric, F.Cu at (105.7, 166.1)
- added C31: DNP, Capacitor_SMD:C_0402_1005Metric, F.Cu at (105.7, 168.1)
- added C32: 100n, Capacitor_SMD:C_0603_1608Metric, F.Cu at (83.7, 167.4)
- added C33: 1u, Capacitor_SMD:C_0603_1608Metric, F.Cu at (83.7, 170.0)
- added C34: 100n, Capacitor_SMD:C_0603_1608Metric, F.Cu at (83.7, 172.5)
- added C35: 100n, Capacitor_SMD:C_0603_1608Metric, F.Cu at (83.7, 175.0)
- added C36: 100n, Capacitor_SMD:C_0603_1608Metric, F.Cu at (83.7, 177.5)
- added C37: 100n, Capacitor_SMD:C_0603_1608Metric, F.Cu at (87.7, 162.4)
- added C38: 10u, Capacitor_SMD:C_0603_1608Metric, F.Cu at (87.7, 164.9)
- added C39: 1u, Capacitor_SMD:C_0603_1608Metric, F.Cu at (87.7, 167.4)
- added C4: 100n, Capacitor_SMD:C_0603_1608Metric, B.Cu at (109.4, 139.8)
- added C40: 100n, Capacitor_SMD:C_0603_1608Metric, F.Cu at (190.9, 82.5)
- added C41: 100n, Capacitor_SMD:C_0603_1608Metric, F.Cu at (80.6, 59.6)
- added C42: 100n, Capacitor_SMD:C_0603_1608Metric, F.Cu at (121.7, 131.3)
- added C43: 1u, Capacitor_SMD:C_0603_1608Metric, F.Cu at (196.3, 48.4)
- added C44: 100n, Capacitor_SMD:C_0603_1608Metric, F.Cu at (190.9, 85.0)
- added C45: 100n, Capacitor_SMD:C_0603_1608Metric, F.Cu at (87.7, 170.0)
- added C46: 100n, Capacitor_SMD:C_0603_1608Metric, F.Cu at (106.6, 105.5)
- added C47: 100n, Capacitor_SMD:C_0603_1608Metric, F.Cu at (196.3, 50.9)
- added C48: 1u, Capacitor_SMD:C_0603_1608Metric, F.Cu at (196.3, 53.4)
- added C49: 1u, Capacitor_SMD:C_0603_1608Metric, F.Cu at (200.3, 38.3)
- added C5: 100n, Capacitor_SMD:C_0603_1608Metric, B.Cu at (101.6, 130.1)
- added C50: 100n, Capacitor_SMD:C_0603_1608Metric, F.Cu at (200.3, 40.8)
- added C51: DNP, Capacitor_SMD:C_0603_1608Metric, F.Cu at (200.3, 43.4)
- added C52: 100n, Capacitor_SMD:C_0603_1608Metric, F.Cu at (188.7, 135.8)
- added C6: 100n, Capacitor_SMD:C_0603_1608Metric, B.Cu at (99.7, 131.9)
- added C7: 100n, Capacitor_SMD:C_0603_1608Metric, B.Cu at (99.6, 137.5)
- added C8: 22p, Capacitor_SMD:C_0603_1608Metric, F.Cu at (96.6, 131.8)
- added C9: 22p, Capacitor_SMD:C_0603_1608Metric, F.Cu at (96.6, 134.9)
- added D1: LED, LED_SMD:LED_0603_1608Metric, F.Cu at (54.0, 116.4)
- added D10: D, Diode_SMD:D_1206_3216Metric, F.Cu at (228.7, 24.2)
- added D2: LED, LED_SMD:LED_0603_1608Metric, F.Cu at (117.8, 135.5)
- added D4: SMAJ5.0A, Diode_SMD:D_SMA, F.Cu at (229.9, 20.2)
- added D5: LED, LED_SMD:LED_0603_1608Metric, F.Cu at (227.9, 33.5)
- added D6: D, Diode_SMD:D_1206_3216Metric_Pad1.42x1.75mm_HandSolder, F.Cu at (98.2, 50.0)
- added D7: D, Diode_SMD:D_1206_3216Metric_Pad1.42x1.75mm_HandSolder, F.Cu at (98.2, 53.4)
- added D8: D, Diode_SMD:D_0805_2012Metric_Pad1.15x1.40mm_HandSolder, F.Cu at (97.6, 56.6)
- added D9: LED, LED_SMD:LED_0603_1608Metric, F.Cu at (106.3, 186.7)
- added F1: RGEF1400, Resistor_THT:R_Axial_DIN0204_L3.6mm_D1.6mm_P5.08mm_Horizontal, F.Cu at (227.3, 30.7)
- added J1: Conn_01x04_Pin, Connector_PinHeader_2.54mm:PinHeader_1x04_P2.54mm_Vertical, F.Cu at (197.0, 134.4)
- added J10: Conn_01x02_Socket, Connector_PinSocket_2.54mm:PinSocket_1x02_P2.54mm_Vertical, F.Cu at (230.9, 39.4)
- added J11: Conn_01x02_Pin, Connector_PinHeader_2.54mm:PinHeader_1x02_P2.54mm_Vertical, F.Cu at (58.0, 153.5)
- added J12: USB_C_Receptacle_USB2.0_14P, Connector_USB:USB_C_Receptacle_Palconn_UTC16-G, F.Cu at (101.1, 28.8)
- added J13: USB_C_Receptacle_USB2.0_14P, Connector_USB:USB_C_Receptacle_Palconn_UTC16-G, F.Cu at (101.1, 38.8)
- added J14: IDC_Cable_02x08, Connector_IDC:IDC-Header_2x08_P2.54mm_Vertical, F.Cu at (71.9, 30.8)
- added J15: Conn_01x02_Pin, Connector_PinHeader_2.54mm:PinHeader_1x02_P2.54mm_Vertical, F.Cu at (92.9, 50.6)
- added J16: Conn_01x04_Pin, Connector_PinHeader_2.54mm:PinHeader_1x04_P2.54mm_Vertical, F.Cu at (84.0, 181.0)
- added J17: Conn_01x04_Pin, Connector_PinHeader_2.54mm:PinHeader_1x04_P2.54mm_Vertical, F.Cu at (88.6, 181.0)
- added J18: Micro_SD_Card, Connector_Card:microSD_HC_Hirose_DM3BT-DSF-PEJS, F.Cu at (87.0, 34.0)
- added J2: Conn_01x02_Socket, Connector_PinSocket_2.54mm:PinSocket_1x02_P2.54mm_Vertical, F.Cu at (201.9, 146.6)
- added J21: MIC_I2S_CONNECTOR, Connector_PinSocket_2.54mm:PinSocket_1x06_P2.54mm_Vertical, F.Cu at (184.4, 134.4)
- added J3: Conn_01x03_Socket, Connector_PinSocket_2.54mm:PinSocket_1x03_P2.54mm_Vertical, F.Cu at (201.6, 134.4)
- added J4: Conn_01x04_Pin, Connector_PinHeader_2.54mm:PinHeader_1x04_P2.54mm_Vertical, F.Cu at (49.0, 148.9)
- added J5: Conn_01x02_Pin, Connector_PinHeader_2.54mm:PinHeader_1x02_P2.54mm_Vertical, F.Cu at (53.0, 153.0)
- added J6: Conn_01x02_Socket, Connector_PinSocket_2.54mm:PinSocket_1x02_P2.54mm_Vertical, F.Cu at (187.2, 96.1)
- added J7: Conn_01x02_Socket, Connector_PinSocket_2.54mm:PinSocket_1x02_P2.54mm_Vertical, F.Cu at (191.8, 96.1)
- added J8: Conn_01x02_Socket, Connector_PinSocket_2.54mm:PinSocket_1x02_P2.54mm_Vertical, F.Cu at (196.4, 96.1)
- added J9: Barrel_Jack, Connector_BarrelJack:BarrelJack_SwitchcraftConxall_RAPC10U_Horizontal, F.Cu at (223.8, 27.5)
- added L1: 1u, Inductor_SMD:L_Bourns-SRN8040_8x8.15mm, F.Cu at (223.7, 42.0)
- added L2: DNP, Inductor_SMD:L_0402_1005Metric, F.Cu at (108.6, 162.2)
- added L3: DNP, Inductor_SMD:L_0402_1005Metric, F.Cu at (108.6, 164.2)
- added L4: 2n, Inductor_SMD:L_0402_1005Metric, F.Cu at (108.6, 166.2)
- added Q1: NMOS, Package_TO_SOT_SMD:TO-252-3_TabPin2, F.Cu at (225.7, 51.0)
- added Q2: NMOS, Package_TO_SOT_SMD:SOT-23, F.Cu at (103.7, 50.5)
- added Q4: AO3400A, Package_TO_SOT_SMD:SOT-23, F.Cu at (197.2, 146.5)
- added Q5: AO3400A, Package_TO_SOT_SMD:SOT-23, F.Cu at (197.2, 151.0)
- added R10: 10k, Resistor_SMD:R_0603_1608Metric, F.Cu at (56.2, 125.0)
- added R11: 330, Resistor_SMD:R_0603_1608Metric, F.Cu at (114.5, 135.5)
- added R12: 0R, Resistor_SMD:R_0603_1608Metric, F.Cu at (105.4, 145.8)
- added R13: 0R, Resistor_SMD:R_0603_1608Metric, F.Cu at (102.6, 145.7)
- added R14: 0R, Resistor_SMD:R_0603_1608Metric, F.Cu at (99.8, 145.7)
- added R15: 10k, Resistor_SMD:R_0603_1608Metric, B.Cu at (101.4, 139.8)
- added R17: 10k, Resistor_SMD:R_0603_1608Metric, F.Cu at (121.7, 135.0)
- added R18: 10k, Resistor_SMD:R_0603_1608Metric, F.Cu at (118.8, 128.2)
- added R19: 1k, Resistor_SMD:R_0603_1608Metric, F.Cu at (121.7, 138.2)
- added R2: 10k, Resistor_SMD:R_0603_1608Metric, F.Cu at (188.7, 138.4)
- added R20: 0R, Resistor_SMD:R_0603_1608Metric, F.Cu at (190.9, 87.5)
- added R21: 2k2, Resistor_SMD:R_0603_1608Metric, F.Cu at (190.9, 90.0)
- added R22: 1k, Resistor_SMD:R_0603_1608Metric, F.Cu at (190.9, 92.6)
- added R23: 18k, Resistor_SMD:R_0603_1608Metric, F.Cu at (194.9, 82.5)
- added R24: 10k, Resistor_SMD:R_0603_1608Metric, F.Cu at (194.9, 85.0)
- added R25: 10k, Resistor_SMD:R_0603_1608Metric, F.Cu at (194.9, 87.5)
- added R26: 1k, Resistor_SMD:R_0603_1608Metric, F.Cu at (194.9, 90.0)
- added R27: 1k, Resistor_SMD:R_0603_1608Metric, F.Cu at (194.9, 92.6)
- added R28: 1k, Resistor_SMD:R_0603_1608Metric, F.Cu at (198.9, 82.5)
- added R29: 1k, Resistor_SMD:R_0603_1608Metric, F.Cu at (198.9, 85.0)
- added R3: 2k2, Resistor_SMD:R_0603_1608Metric, F.Cu at (188.7, 140.9)
- added R30: 210k, Resistor_SMD:R_0603_1608Metric, F.Cu at (198.9, 87.5)
- added R31: 10R, Resistor_SMD:R_0603_1608Metric, F.Cu at (200.3, 45.9)
- added R32: 10k, Resistor_SMD:R_0603_1608Metric, F.Cu at (200.3, 48.4)
- added R33: 2m, Resistor_SMD:R_0603_1608Metric, F.Cu at (200.3, 50.9)
- added R34: 0R, Resistor_SMD:R_0603_1608Metric, F.Cu at (198.9, 90.0)
- added R35: 0R, Resistor_SMD:R_0603_1608Metric, F.Cu at (198.9, 92.6)
- added R36: 100k, Resistor_SMD:R_0603_1608Metric, F.Cu at (188.7, 143.4)
- added R37: 1k, Resistor_SMD:R_0603_1608Metric, F.Cu at (121.7, 128.1)
- added R38: 10k, Resistor_SMD:R_0603_1608Metric, F.Cu at (200.3, 53.4)
- added R39: 10k, Resistor_SMD:R_0603_1608Metric, F.Cu at (204.4, 38.3)
- added R4: 330, Resistor_SMD:R_0603_1608Metric, F.Cu at (61.8, 119.0)
- added R40: 453k, Resistor_SMD:R_0603_1608Metric, F.Cu at (204.4, 40.8)
- added R41: 100k, Resistor_SMD:R_0603_1608Metric, F.Cu at (204.4, 43.4)
- added R42: 2m, Resistor_SMD:R_0603_1608Metric, F.Cu at (204.4, 45.9)
- added R43: 330, Resistor_SMD:R_0603_1608Metric, F.Cu at (204.4, 48.4)
- added R44: 5k1, Resistor_SMD:R_0603_1608Metric, F.Cu at (80.6, 62.1)
- added R45: 5k1, Resistor_SMD:R_0603_1608Metric, F.Cu at (84.6, 49.5)
- added R46: 5k1, Resistor_SMD:R_0603_1608Metric, F.Cu at (84.6, 52.0)
- added R47: 5k1, Resistor_SMD:R_0603_1608Metric, F.Cu at (84.6, 54.5)
- added R48: 22R, Resistor_SMD:R_0603_1608Metric, F.Cu at (84.6, 57.1)
- added R49: 22R, Resistor_SMD:R_0603_1608Metric, F.Cu at (84.6, 59.6)
- added R5: 5k1, Resistor_SMD:R_0603_1608Metric, F.Cu at (53.2, 130.0)
- added R50: 22R, Resistor_SMD:R_0603_1608Metric, F.Cu at (84.6, 62.1)
- added R51: 22R, Resistor_SMD:R_0603_1608Metric, F.Cu at (88.6, 49.5)
- added R52: 10R, Resistor_SMD:R_0603_1608Metric, F.Cu at (88.6, 52.0)
- added R53: 10k, Resistor_SMD:R_0603_1608Metric, F.Cu at (88.6, 54.5)
- added R54: 330, Resistor_SMD:R_0603_1608Metric, F.Cu at (87.7, 172.5)
- added R55: 0R, Resistor_SMD:R_0603_1608Metric, F.Cu at (87.7, 175.0)
- added R56: 0R, Resistor_SMD:R_0603_1608Metric, F.Cu at (87.7, 177.5)
- added R57: 0R, Resistor_SMD:R_0603_1608Metric, F.Cu at (91.7, 162.4)
- added R58: 0R, Resistor_SMD:R_0603_1608Metric, F.Cu at (91.7, 164.9)
- added R59: 10k, Resistor_SMD:R_0603_1608Metric, F.Cu at (91.7, 167.4)
- added R6: 5k1, Resistor_SMD:R_0603_1608Metric, F.Cu at (50.0, 130.0)
- added R60: 10k, Resistor_SMD:R_0603_1608Metric, F.Cu at (91.7, 170.0)
- added R61: DNP, Resistor_SMD:R_0603_1608Metric, F.Cu at (88.6, 57.1)
- added R62: DNP, Resistor_SMD:R_0603_1608Metric, F.Cu at (88.6, 59.6)
- added R68: DNP, Resistor_SMD:R_0603_1608Metric, F.Cu at (204.4, 50.9)
- added R69: 0R, Resistor_SMD:R_0603_1608Metric, F.Cu at (204.4, 53.4)
- added R7: 10k, Resistor_SMD:R_0603_1608Metric, F.Cu at (111.0, 112.3)
- added R70: 0R, Resistor_SMD:R_0603_1608Metric, F.Cu at (208.4, 38.3)
- added R71: DNP, Resistor_SMD:R_0603_1608Metric, F.Cu at (208.4, 40.8)
- added R72: DNP, Resistor_SMD:R_0603_1608Metric, F.Cu at (208.4, 43.4)
- added R73: 0R, Resistor_SMD:R_0603_1608Metric, F.Cu at (208.4, 45.9)
- added R74: DNP, Resistor_SMD:R_0603_1608Metric, F.Cu at (208.4, 48.4)
- added R75: 0R, Resistor_SMD:R_0603_1608Metric, F.Cu at (208.4, 50.9)
- added R76: 1k, Resistor_SMD:R_0603_1608Metric, F.Cu at (91.7, 172.5)
- added R78: 10k, Resistor_SMD:R_0603_1608Metric, F.Cu at (91.7, 175.0)
- added R79: 10k, Resistor_SMD:R_0603_1608Metric, F.Cu at (91.7, 177.5)
- added R8: 10k, Resistor_SMD:R_0603_1608Metric, F.Cu at (114.0, 112.3)
- added R80: 10, Resistor_SMD:R_0603_1608Metric, F.Cu at (188.7, 145.9)
- added R81: 10k, Resistor_SMD:R_0603_1608Metric, F.Cu at (192.7, 133.3)
- added R82: 17, Resistor_SMD:R_0603_1608Metric, F.Cu at (192.7, 135.8)
- added R83: 10, Resistor_SMD:R_0603_1608Metric, F.Cu at (192.7, 138.4)
- added R84: 10k, Resistor_SMD:R_0603_1608Metric, F.Cu at (192.7, 140.9)
- added R85: 17, Resistor_SMD:R_0603_1608Metric, F.Cu at (192.7, 143.4)
- added R9: 7k, Resistor_SMD:R_0603_1608Metric, F.Cu at (46.2, 127.0)
- added SW2: SW_Push, Button_Switch_THT:SW_PUSH_6mm, F.Cu at (124.3, 137.2)
- added SW5: SW_Push, Button_Switch_THT:SW_PUSH_6mm, F.Cu at (124.4, 127.2)
- added SW6: SW_Push, Button_Switch_THT:SW_PUSH_6mm, F.Cu at (95.8, 163.2)
- added SW7: SW_Push, Button_Switch_THT:SW_PUSH_6mm, F.Cu at (95.8, 171.8)
- added TSAL2: LED, LED_SMD:LED_0603_1608Metric, F.Cu at (188.7, 148.4)
- added TSAL3: LED, LED_SMD:LED_0603_1608Metric, F.Cu at (188.7, 151.0)
- added U1: TMP117xxDRV, Package_SON:WSON-6-1EP_2x2mm_P0.65mm_EP1x1.6mm, F.Cu at (192.6, 149.0)
- added U10: INA219AxD, Package_SO:SOIC-8_3.9x4.9mm_P1.27mm, F.Cu at (214.6, 47.0)
- added U11: TLV62569ADRL, Package_TO_SOT_SMD:SOT-563, F.Cu at (227.6, 27.6)
- added U12: USBLC6-2P6, Package_TO_SOT_SMD:SOT-666, F.Cu at (92.7, 57.2)
- added U13: USBLC6-2P6, Package_TO_SOT_SMD:SOT-666, F.Cu at (92.7, 60.7)
- added U14: ESP32-C3FH4, Package_DFN_QFN:QFN-32-1EP_5x5mm_P0.5mm_EP3.45x3.45mm, F.Cu at (108.3, 172.7)
- added U15: TPS60400DBV, Package_TO_SOT_SMD:SOT-23-5, F.Cu at (212.9, 52.6)
- added U16: TLV172IDCK, Package_TO_SOT_SMD:SOT-353_SC-70-5, F.Cu at (202.9, 90.1)
- added U2: RV-3028-C7, Package_SON:MicroCrystal_C7_SON-8_1.5x3.2mm_P0.9mm, F.Cu at (113.0, 105.3)
- added U3: STM32G474RETx, Package_QFP:LQFP-64_10x10mm_P0.5mm, F.Cu at (105.4, 134.9)
- added U5: MAX98357A, Package_DFN_QFN:TQFN-16-1EP_3x3mm_P0.5mm_EP1.23x1.23mm, F.Cu at (201.7, 96.4)
- added U6: TLV172IDCK, Package_TO_SOT_SMD:SOT-353_SC-70-5, F.Cu at (202.9, 83.1)
- added U7: TLV172IDCK, Package_TO_SOT_SMD:SOT-353_SC-70-5, F.Cu at (202.9, 86.6)
- added U8: MAX98357A, Package_DFN_QFN:TQFN-16-1EP_3x3mm_P0.5mm_EP1.23x1.23mm, F.Cu at (201.7, 101.7)
- added U9: INA219AxD, Package_SO:SOIC-8_3.9x4.9mm_P1.27mm, F.Cu at (214.6, 40.4)
- added Y1: 16MHz, Crystal:Crystal_SMD_ECS_CSM3X-2Pin_7.6x4.1mm, F.Cu at (92.0, 133.3)
- added Y2: 40MHz, Crystal:Crystal_SMD_ECS_CSM3X-2Pin_7.6x4.1mm, F.Cu at (99.0, 188.2)
Routing:
- net 3V3: track 0.00 -> 30.2 mm, vias 0 -> 6
- net /STM32G4/CLK_OUT: track 0.00 -> 9.67 mm
- net /STM32G4/CLK_IN: track 0.00 -> 9.18 mm
- net Net-(U3-PA4): track 0.00 -> 3.03 mm, vias 0 -> 1

Commit message: PCB Work
Parts:
- C32, C33, C34, C35, C36, C37, C38, C39, R10, R5, R6, R9: moved to B.Cu
- L4: footprint Inductor_SMD:L_0402_1005Metric -> Inductor_SMD:L_0603_1608Metric_Pad1.05x0.95mm_HandSolder; moved to B.Cu
- moved R8 85.1 mm to (45.3, 62.2)
- moved R7 84.2 mm to (45.3, 59.7)
- moved U2 78.9 mm to (49.4, 58.6)
- moved C46 78.1 mm to (45.3, 57.2)
- moved J4 74.6 mm to (114.3, 112.7), turned to 90 degrees
- moved R9 62.3 mm to (108.0, 135.1), turned to 90 degrees
- moved R5 58.1 mm to (111.0, 135.0), turned to -90 degrees
- moved R6 56.3 mm to (106.3, 131.9), turned to -90 degrees
- moved J5 54.0 mm to (86.5, 110.7)
- moved R10 52.2 mm to (108.0, 131.9), turned to 90 degrees
- moved AE1 50.3 mm to (57.9, 172.0), turned to 90 degrees
- moved L2 49.3 mm to (60.3, 172.0)
- moved C28 48.0 mm to (58.9, 172.5), turned to -90 degrees
- moved L3 45.1 mm to (64.2, 172.1)
- moved C29 44.7 mm to (61.8, 172.5), turned to -90 degrees
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Connections:
- net /STM32G4/INT_RTC renamed /Peripherials/INT_RTC
- J17 pad 2: /ESP32C3/BOOT -> /ESP32C3/GPIO8
- J17 pad 3: /ESP32C3/GPIO8 -> /ESP32C3/BOOT
Routing:
- net /ESP32C3/SPI1_MISO: track 0.00 -> 43.5 mm, vias 0 -> 1
- net /STM32G4/nRST: track 0.00 -> 43.0 mm
- net /STM32G4/BOOT0: track 0.00 -> 24.8 mm
- net /ESP32C3/BOOT: track 0.00 -> 23.2 mm
- net /STM32G4/SWDIO: track 0.00 -> 21.8 mm
- net /STM32G4/SWDCLK: track 0.00 -> 20.9 mm
- net 3V3: track 30.2 -> 50.4 mm, vias 6 -> 11
- net /ESP32C3/SPI1_MOSI: track 0.00 -> 18.1 mm, vias 0 -> 1
- net /ESP32C3/SPI1_SCLK: track 0.00 -> 17.7 mm, vias 0 -> 1
- net /ESP32C3/ESP32_RST: track 0.00 -> 15.2 mm
- net /ESP32C3/GPIO8: track 0.00 -> 15.1 mm
- net Net-(R18-Pad2): track 0.00 -> 12.1 mm
- net /ESP32C3/SPI1_CS_ESP: track 0.00 -> 10.9 mm
- net Net-(R76-Pad2): track 0.00 -> 10.7 mm
- net Net-(R17-Pad1): track 0.00 -> 10.6 mm
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Other:
- copper layers 2 -> 4

Commit message: Basic STM + ESP Routing
Parts:
- moved J14 158.8 mm to (117.3, 182.9), turned to -90 degrees
- moved J4 77.2 mm to (134.4, 187.2), turned to -90 degrees
- moved J5 58.7 mm to (132.1, 147.8), turned to -90 degrees
- moved SW2 50.9 mm to (123.8, 166.3), turned to 0 degrees
- moved C11 50.2 mm to (121.2, 170.4), turned to -90 degrees
- moved R19 48.1 mm to (121.2, 167.2), turned to 90 degrees
- moved SW5 47.1 mm to (123.9, 156.2), turned to 0 degrees
- moved R17 46.3 mm to (121.2, 164.0), turned to 90 degrees
- moved C42 44.6 mm to (121.2, 160.3), turned to -90 degrees
- moved R37 43.6 mm to (121.2, 157.1), turned to 90 degrees
- moved D2 41.0 mm to (110.0, 175.8), turned to -90 degrees
- moved R11 40.8 mm to (107.3, 175.7), turned to -90 degrees
- moved C10 40.4 mm to (111.7, 171.4), turned to 90 degrees
- moved R18 39.6 mm to (118.3, 157.2), turned to 90 degrees
- moved R10 37.4 mm to (110.9, 169.2), turned to 0 degrees
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Connections:
- U3 pad 30: /Peripherials/MATRIX_A -> /Peripherials/MATRIX_D
- U3 pad 33: /Peripherials/MATRIX_C -> /Peripherials/MATRIX_LAT
- U3 pad 56: /Peripherials/MATRIX_D -> /Peripherials/MATRIX_A
- U3 pad 57: /Peripherials/MATRIX_LAT -> /Peripherials/MATRIX_C
- U3 pad 58: /Peripherials/MATRIX_R1 -> /Peripherials/MATRIX_R2
- U3 pad 59: /Peripherials/MATRIX_B1 -> /Peripherials/MATRIX_R1
- U3 pad 60: /Peripherials/MATRIX_R2 -> /Peripherials/MATRIX_B2
- U3 pad 62: /Peripherials/MATRIX_B2 -> /Peripherials/MATRIX_B1
Routing:
- net /Peripherials/MATRIX_B1: track 0.00 -> 29.8 mm, vias 0 -> 1
- net /Peripherials/MATRIX_B2: track 0.00 -> 28.5 mm, vias 0 -> 1
- net /Peripherials/MATRIX_G2: track 0.00 -> 24.8 mm
- net /Peripherials/MATRIX_G1: track 0.00 -> 24.4 mm
- net /Peripherials/MATRIX_B: track 0.00 -> 23.2 mm
- net /Peripherials/MATRIX_C: track 0.00 -> 23.1 mm, vias 0 -> 1
- net /Peripherials/MATRIX_R1: track 0.00 -> 21.7 mm, vias 0 -> 1
- net /Peripherials/MATRIX_R2: track 0.00 -> 21.1 mm, vias 0 -> 1
- net /Peripherials/MATRIX_A: track 0.00 -> 18.9 mm, vias 0 -> 1
- net /Peripherials/MATRIX_D: track 0.00 -> 18.1 mm
- net /Peripherials/MATRIX_OE: track 0.00 -> 14.8 mm
- net /Peripherials/MATRIX_LAT: track 0.00 -> 14.4 mm
- net /STM32G4/nRST: track 43.0 -> 55.2 mm
- net /STM32G4/BOOT0: track 24.8 -> 33.9 mm
- net /STM32G4/SWDCLK: track 20.9 -> 25.7 mm
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
Commit message: Pin swaps
Parts:
- removed TSAL2, TSAL3: LED, LED_SMD:LED_0603_1608Metric
- C12, C13, C16, C17, C41, R44, R45, R46, R47, R61, R62: moved to B.Cu
- moved C46 173.2 mm to (206.7, 119.9)
- moved R7 173.2 mm to (206.7, 122.4)
- moved R8 173.2 mm to (206.7, 124.9)
- moved U2 173.2 mm to (210.8, 121.3)
- moved J13 98.0 mm to (67.6, 124.5)
- moved J12 97.4 mm to (80.9, 124.5)
- moved Q2 92.2 mm to (31.4, 107.8)
- moved D6 90.5 mm to (64.8, 134.1), turned to 90 degrees
- moved J18 88.9 mm to (96.5, 119.4)
- moved J15 87.1 mm to (26.8, 107.3)
- moved R52 87.1 mm to (22.5, 108.7)
- moved D8 87.1 mm to (31.6, 113.3)
- moved R53 87.1 mm to (22.5, 111.3)
- moved D7 83.2 mm to (78.0, 134.1), turned to 90 degrees
- moved R51 83.1 mm to (66.9, 129.8), turned to -90 degrees
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Routing:
- net /Analog/I2S2_WS: track 0.00 -> 18.0 mm, vias 0 -> 2
- net Net-(J13-SHIELD): track 0.00 -> 17.3 mm
- net Net-(J12-SHIELD): track 0.00 -> 17.3 mm
- net /Analog/I2S2_CK: track 0.00 -> 17.0 mm, vias 0 -> 2
- net /Analog/I2S2_SD: track 0.00 -> 15.3 mm, vias 0 -> 2
- net 3V3: track 50.4 -> 63.6 mm, vias 11 -> 14
- net /Peripherials/VBUS_STM: track 0.00 -> 11.5 mm, vias 0 -> 2
- net /Peripherials/VBUS_ESP: track 0.00 -> 11.4 mm, vias 0 -> 2
- net /Peripherials/USB_P_ESP_RES: track 0.00 -> 4.43 mm
- net /Peripherials/USB_N_STM_RES: track 0.00 -> 4.41 mm
- net /Peripherials/USB_N_ESP_RES: track 0.00 -> 4.40 mm
- net /Peripherials/USB_P_STM_RES: track 0.00 -> 4.26 mm
- net Net-(J7-Pin_1): track 0.00 -> 3.58 mm
- net Net-(J7-Pin_2): track 0.00 -> 3.57 mm
- net Net-(J8-Pin_1): track 0.00 -> 3.06 mm
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Other:
- board text added: "STM32G474"

Commit message: PCB Grouping Work
Parts:
- added J19: Conn_01x02_Socket, Connector_PinSocket_2.54mm:PinSocket_1x02_P2.54mm_Vertical, F.Cu at (181.6, 146.5)
- added J20: Conn_01x02_Socket, Connector_PinSocket_2.54mm:PinSocket_1x02_P2.54mm_Vertical, F.Cu at (185.1, 125.1)
- C14, R2, R3, R36, R82: moved to B.Cu
- moved R2 80.1 mm to (262.5, 109.8), turned to 180 degrees
- moved U1 77.1 mm to (262.5, 109.8)
- moved R36 54.2 mm to (260.5, 95.3), turned to -90 degrees
- moved J3 53.1 mm to (263.1, 91.9)
- moved R3 35.6 mm to (262.1, 146.1), turned to -90 degrees
- moved J2 33.3 mm to (264.8, 146.6)
- moved R82 14.2 mm to (184.2, 146.5), turned to 180 degrees
- moved J1 13.2 mm to (263.7, 126.3)
- moved R81 10.1 mm to (171.8, 147.4), turned to 180 degrees
- moved C14 8.42 mm to (260.4, 133.8), turned to 180 degrees
- moved R80 5.99 mm to (171.8, 145.5), turned to 180 degrees
- moved Q4 4.07 mm to (175.3, 146.5)
Routing:
- net Net-(Q4-G): track 0.00 -> 3.64 mm
- net Net-(J19-Pin_2): track 0.00 -> 2.86 mm
- net /STM32G4/ALS_ADC: track 0.00 -> 2.80 mm
- net /STM32G4/PAPIR: track 0.00 -> 2.66 mm
- net 3V3: track 63.6 -> 66.2 mm
- net /STM32G4/INT_TEMP_ALERT: track 0.00 -> 2.16 mm, vias 0 -> 1
- net Net-(J19-Pin_1): track 0.00 -> 1.80 mm
Other:
- board text added: "3V3"
- board text added: "ALS"
- board text added: "EXTERNAL I2C TEMP"
- board text added: "GND"
- board text added: "INTERNAL I2C TEMP"
- board text added: "PIR"
- board text added: "PIR SENSOR"
- board text added: "SCL"
- board text added: "SDA"
- board text added: "SPEAKER DAC"

Commit message: Almost Done with Dev Board
Parts:
- removed D1: LED, LED_SMD:LED_0603_1608Metric
- removed J11: Conn_01x02_Pin, Connector_PinHeader_2.54mm:PinHeader_1x02_P2.54mm_Vertical
- removed R4: 330, Resistor_SMD:R_0603_1608Metric
- added C53: 100n, Capacitor_SMD:C_0603_1608Metric, B.Cu at (87.7, 90.6)
- C14, R3, R36: moved to F.Cu
- C18, C19, C40, C43, C44, C46, R7, R8, R85: moved to B.Cu
- R33: footprint Resistor_SMD:R_0603_1608Metric -> Resistor_SMD:R_1206_3216Metric
- moved J2 186.1 mm to (90.5, 81.4), turned to 90 degrees
- moved R3 183.0 mm to (90.0, 84.0), turned to 0 degrees
- moved J7 178.8 mm to (60.4, 124.4), turned to 90 degrees
- moved C13 173.3 mm to (61.9, 120.5), turned to 90 degrees
- moved U5 173.1 mm to (62.2, 120.5), turned to -90 degrees
- moved C12 171.9 mm to (63.5, 120.5), turned to 90 degrees
- moved R20 171.8 mm to (60.4, 117.5), turned to 0 degrees
- moved J8 171.5 mm to (68.2, 124.4), turned to 90 degrees
- moved C17 169.0 mm to (67.0, 121.1), turned to 90 degrees
- moved R35 168.8 mm to (63.5, 117.5), turned to 180 degrees
- moved C16 167.6 mm to (68.6, 121.1), turned to 90 degrees
- moved J3 166.4 mm to (97.0, 81.3), turned to 90 degrees
- moved U8 165.6 mm to (70.1, 120.5), turned to -90 degrees
- moved R30 164.2 mm to (68.4, 117.6), turned to 0 degrees
- moved J1 164.0 mm to (106.0, 81.4), turned to 90 degrees
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Connections:
- Q1 pad 1: Net-(J10-Pin_2) -> Net-(Q1-G)
- Q1 pad 2: Net-(Q1-G) -> Net-(J10-Pin_2)
- U3 pad 10: /Analog/LEFT_SD_MODE -> /Analog/RIGHT_SD_MODE
- U3 pad 11: /Analog/RIGHT_SD_MODE -> /Analog/LEFT_SD_MODE
Routing:
- net /ESP32C3/SPI1_MOSI: track 18.1 -> 87.2 mm, vias 1 -> 4
- net /ESP32C3/SPI1_MISO: track 43.5 -> 110.2 mm, vias 1 -> 4
- net /ESP32C3/SPI1_SCLK: track 17.7 -> 79.9 mm, vias 1 -> 4
- net /ESP32C3/SPI1_CS_ESP: track 10.9 -> 71.8 mm, vias 0 -> 2
- net /Analog/LEFT_SD_MODE: track 0.00 -> 57.5 mm, vias 0 -> 2
- net /Power/MATRIX_PWR_EN: track 0.00 -> 56.6 mm, vias 0 -> 4
- net /Power/I2C3_SCL: track 3.39 -> 56.5 mm, vias 1 -> 2
- net /STM32G4/TV_IR_PWM_1: track 0.00 -> 51.7 mm, vias 0 -> 2
- net /Analog/RIGHT_SD_MODE: track 0.00 -> 49.5 mm, vias 0 -> 2
- net /STM32G4/TV_IR_PWM_2: track 0.00 -> 48.5 mm, vias 0 -> 2
- net /Power/I2C3_SDA: track 4.19 -> 50.4 mm, vias 1 -> 2
- net /STM32G4/I2S3_CK: track 0.00 -> 43.7 mm, vias 0 -> 1
- net /STM32G4/I2S3_WS: track 0.00 -> 42.8 mm, vias 0 -> 1
- net /STM32G4/I2S3_SD: track 0.00 -> 41.0 mm, vias 0 -> 1
- net /Peripherials/FAN_PWM: track 0.00 -> 40.8 mm, vias 0 -> 2
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Other:
- board outline added: 128.7 x 50.4 mm
- board text added: "A"
- board text added: "BOOT0"
- board text added: "CK"
- board text added: "DISPLAY"
- board text added: "FAN"
- board text added: "K"
- board text added: "MIC"
- board text added: "NRST"
- board text added: "PWR"
- board text added: "RTC"
- board text added: "SD"
- board text added: "SPEAKER DACs"
- board text added: "SWCLK"
- board text added: "SWDIO"
- board text added: "TEMP"
- board text added: "WS"
- board text removed: "EXTERNAL I2C TEMP"
- board text removed: "INTERNAL I2C TEMP"
- board text removed: "PIR SENSOR"
- board text removed: "SPEAKER DAC"

Commit message: DONE?? (Minor fixes needed)
Parts:
- added C54: DNP, Capacitor_SMD:C_0603_1608Metric, F.Cu at (145.8, 100.6)
- added C55: DNP, Capacitor_SMD:C_0603_1608Metric, F.Cu at (144.3, 100.6)
- C43: moved to F.Cu
- R72, R73, R74, R75: moved to B.Cu
- moved D5 56.0 mm to (143.5, 90.9), turned to 180 degrees
- moved R43 52.9 mm to (140.5, 90.9)
- moved C19 51.1 mm to (142.5, 92.7), turned to 0 degrees
- moved D10 50.7 mm to (141.2, 108.0), turned to 180 degrees
- moved R42 50.0 mm to (139.7, 96.0), turned to 90 degrees
- moved L1 44.2 mm to (151.4, 102.6), turned to 90 degrees
- moved R40 43.8 mm to (142.7, 100.6), turned to -90 degrees
- moved R41 43.7 mm to (142.7, 103.6), turned to -90 degrees
- moved U11 43.0 mm to (145.0, 103.9)
- moved U10 42.2 mm to (144.3, 94.7), turned to 180 degrees
- moved C51 42.2 mm to (141.2, 100.6), turned to -90 degrees
- moved C21 40.8 mm to (139.7, 100.6), turned to -90 degrees
- moved R75 34.9 mm to (146.3, 96.8)
- moved C20 34.8 mm to (143.3, 105.9), turned to 180 degrees
- moved R72 30.7 mm to (150.3, 96.8)
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Connections:
- AE1 pad 2: (no net) -> GND
Routing:
- net USB_5V: track 0.00 -> 99.7 mm, vias 0 -> 6
- net 5V: track 10.2 -> 98.9 mm, vias 0 -> 12
- net -3V3: track 3.27 -> 89.2 mm, vias 0 -> 3
- net /Power/I2C3_SCL: track 56.5 -> 110.3 mm, vias 2 -> 3
- net /Power/5V_VOLTS: track 0.00 -> 46.4 mm, vias 0 -> 2
- net 3V3: track 86.7 -> 130.2 mm, vias 19 -> 35
- net /Power/I2C3_SDA: track 50.4 -> 93.8 mm
- net /Peripherials/INT_RTC: track 3.48 -> 34.8 mm, vias 1 -> 2
- net /Peripherials/VBUS_STM: track 11.5 -> 31.4 mm, vias 2 -> 3
- net /ESP32C3/SPI1_MISO: track 110.2 -> 99.8 mm
- net Net-(R76-Pad2): track 20.5 -> 10.7 mm
- net Net-(U10-A1): track 0.00 -> 4.86 mm, vias 0 -> 1
- net Net-(U11-FB): track 0.00 -> 4.76 mm
- net Net-(U10-A0): track 0.00 -> 4.58 mm, vias 0 -> 1
- net Net-(F1-Pad1): track 7.81 -> 3.63 mm
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- added copper zone on F.Cu, net /Power/3V3_AMPS_1
- added copper zone on In2.Cu, net 3V3
- added copper zone on F.Cu, net 5V
- added copper zone on In2.Cu, net 5V
- added copper zone on B.Cu, net GND
- added copper zone on F.Cu, net GND
- added copper zone on In1.Cu, net GND
- added copper zone on F.Cu, net Net-(U11-SW)
- added copper zone on F.Cu, net USB_5V
Other:
- board size 128.7 x 50.4 mm -> 128.2 x 50.4 mm
