File: SeniorDesign_PCB.kicad_pcb (KiCad board)
At the start: 4 copper layers, 225 parts, among them J1 Conn_01x04_Pin, J10 Conn_01x02_Socket, J11 Conn_01x02_Pin, J12 USB_C_Receptacle_USB2.0_14P, J13 USB_C_Receptacle_USB2.0_14P, J14 IDC_Cable_02x08, J15 Conn_01x02_Pin, J16 Conn_01x04_Pin, J17 Conn_01x04_Pin, J18 Micro_SD_Card, J19 Conn_01x02_Socket, J2 Conn_01x02_Socket, J20 Conn_01x02_Socket, J21 MIC_I2S_CONNECTOR, J22 Conn_01x02_Socket, J23 Conn_01x02_Socket, J24 Conn_01x02_Socket, J25 Conn_01x02_Socket, J26 Conn_01x08_Socket, J27 Conn_01x02_Socket, J3 Conn_01x03_Socket, J4 Conn_01x04_Pin, J5 Conn_01x02_Pin, J6 Conn_01x02_Socket, J7 Conn_01x02_Socket, J8 Conn_01x02_Socket, J9 Conn_01x08_Socket, Q1 NMOS, Q2 NMOS, Q4 AO3400A, Q5 AO3400A, Q6 NMOS, Q7 NMOS, SW2 SW_Push, SW5 SW_Push, SW6 SW_Push, SW7 SW_Push, U1 TMP117xxDRV, U10 INA219AxD, U12 USBLC6-2P6, U13 USBLC6-2P6, U14 ESP32-C3FH4, U15 TPS60400DBV, U16 TLV172IDCK, U17 TCPP03-M20, U18 TPS54302, U2 RV-3028-C7, U3 STM32G474RETx, U4 TPS513885VABR, U5 MAX98357A, U6 TLV172IDCK, U7 TLV172IDCK, U8 MAX98357A, U9 INA219AxD, Y1 16MHz, Y2 40MHz

Commit message: shunts
Parts:
- removed R38, R39: 10k, Resistor_SMD:R_0603_1608Metric
- moved C9 189.8 mm to (142.2, 142.4), turned to -90 degrees
- moved C8 187.5 mm to (140.6, 139.8), turned to 90 degrees
- moved U9 181.6 mm to (37.7, -94.5)
- moved U10 158.3 mm to (63.1, -94.4)
- moved R70 155.0 mm to (32.4, -93.2), turned to 90 degrees
- moved R68 154.7 mm to (32.4, -96.2), turned to 90 degrees
- moved R69 153.4 mm to (34.6, -98.8), turned to 180 degrees
- moved R71 151.6 mm to (37.6, -98.8), turned to 180 degrees
- moved R72 132.4 mm to (57.6, -97.0), turned to 90 degrees
- moved R73 132.3 mm to (57.6, -93.8), turned to 90 degrees
- moved C19 131.7 mm to (42.4, -92.8), turned to 90 degrees
- moved R74 130.6 mm to (60.4, -98.6), turned to 180 degrees
- moved R75 128.1 mm to (63.4, -98.6), turned to 180 degrees
- moved R32 117.2 mm to (170.2, 30.1), turned to 90 degrees
- moved R31 115.7 mm to (168.6, 31.7), turned to 90 degrees
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Routing:
- net Net-(J24-Pin_2): track 0.00 -> 22.3 mm
- net Net-(J10-Pin_1): track 0.00 -> 21.5 mm
- net GND: track 34.0 -> 49.2 mm, vias 34 -> 44
- net 3V3: track 53.9 -> 67.6 mm, vias 12 -> 18
- net /Power/5V_AMPS_1: track 0.00 -> 12.2 mm
- net Net-(Q1-G): track 0.00 -> 6.60 mm
- net Net-(U10-A0): track 0.00 -> 4.68 mm
- net Net-(U9-A0): track 0.00 -> 4.26 mm
- net Net-(U10-A1): track 0.00 -> 3.96 mm
- net Net-(U9-A1): track 0.00 -> 3.83 mm
- net 5V: track 0.00 -> 3.59 mm
