File: SeniorDesign_PCB.kicad_pcb (KiCad board)
At the start: 4 copper layers, 223 parts, among them J1 Conn_01x04_Pin, J10 Conn_01x02_Socket, J11 Conn_01x02_Pin, J12 USB_C_Receptacle_USB2.0_14P, J13 USB_C_Receptacle_USB2.0_14P, J14 IDC_Cable_02x08, J15 Conn_01x02_Pin, J16 Conn_01x04_Pin, J17 Conn_01x04_Pin, J18 Micro_SD_Card, J19 Conn_01x02_Socket, J2 Conn_01x02_Socket, J20 Conn_01x02_Socket, J21 MIC_I2S_CONNECTOR, J22 Conn_01x02_Socket, J23 Conn_01x02_Socket, J24 Conn_01x02_Socket, J25 Conn_01x02_Socket, J26 Conn_01x08_Socket, J27 Conn_01x02_Socket, J3 Conn_01x03_Socket, J4 Conn_01x04_Pin, J5 Conn_01x02_Pin, J6 Conn_01x02_Socket, J7 Conn_01x02_Socket, J8 Conn_01x02_Socket, J9 Conn_01x08_Socket, Q1 NMOS, Q2 NMOS, Q4 AO3400A, Q5 AO3400A, Q6 NMOS, Q7 NMOS, SW2 SW_Push, SW5 SW_Push, SW6 SW_Push, SW7 SW_Push, U1 TMP117xxDRV, U10 INA219AxD, U12 USBLC6-2P6, U13 USBLC6-2P6, U14 ESP32-C3FH4, U15 TPS60400DBV, U16 TLV172IDCK, U17 TCPP03-M20, U18 TPS54302, U2 RV-3028-C7, U3 STM32G474RETx, U4 TPS513885VABR, U5 MAX98357A, U6 TLV172IDCK, U7 TLV172IDCK, U8 MAX98357A, U9 INA219AxD, Y1 16MHz, Y2 40MHz

Commit message: grouped together
Parts:
- moved J4 246.7 mm to (153.6, 119.8), turned to 180 degrees
- moved R5 242.1 mm to (169.2, 125.9)
- moved R6 242.1 mm to (169.2, 128.4)
- moved R19 214.8 mm to (120.4, 53.2), turned to -90 degrees
- moved SW2 213.6 mm to (119.5, 62.8)
- moved C11 212.1 mm to (118.8, 53.2), turned to -90 degrees
- moved R17 206.5 mm to (122.0, 53.2), turned to 90 degrees
- moved C53 123.0 mm to (109.4, 146.4)
- moved R2 17.8 mm to (142.6, -58.6), turned to -90 degrees
- moved R18 12.8 mm to (-47.6, 146.0), turned to 180 degrees
- moved Q4 1.54 mm to (137.2, -96.6)
- moved R80 1.54 mm to (134.7, -93.9)
- moved R81 1.54 mm to (137.3, -93.7)
- moved Q5 1.41 mm to (148.2, -96.6)
- moved R83 1.41 mm to (145.7, -94.1)
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Routing:
- net Net-(J19-Pin_2): track 0.00 -> 5.93 mm
- net Net-(J20-Pin_2): track 0.00 -> 5.91 mm
- net Net-(J19-Pin_1): track 0.00 -> 5.58 mm
- net Net-(J20-Pin_1): track 0.00 -> 5.57 mm
- net Net-(Q4-G): track 0.00 -> 4.09 mm
- net Net-(Q5-G): track 0.00 -> 3.99 mm
- net 3V3: track 67.6 -> 71.5 mm, vias 18 -> 20
- net GND: track 49.2 -> 50.9 mm, vias 44 -> 46

Commit message: rtc, fan, we should fix usb power oring
Parts:
- moved C41 244.7 mm to (166.6, 167.6)
- moved U2 106.8 mm to (8.35, 3.05)
- moved C46 93.2 mm to (10.6, 1.60), turned to 90 degrees
- moved R7 82.6 mm to (10.6, 4.60), turned to 90 degrees
- moved R8 80.8 mm to (6.00, 1.62), turned to -90 degrees
- moved Q2 64.3 mm to (-27.4, 32.3), turned to -90 degrees
- moved D8 59.0 mm to (-26.6, 29.3), turned to 180 degrees
- moved J15 55.0 mm to (-29.5, 23.6)
- moved R53 32.5 mm to (-30.4, 29.3)
- moved R52 31.5 mm to (-30.2, 32.0), turned to -90 degrees
Routing:
- net Net-(D8-A): track 0.00 -> 9.06 mm
- net 3V3: track 71.5 -> 78.0 mm, vias 20 -> 24
- net 5V: track 3.59 -> 9.84 mm
- net GND: track 50.9 -> 57.1 mm, vias 46 -> 49
- net Net-(Q2-G): track 0.00 -> 4.55 mm
- net /Peripherials/INT_RTC: track 0.00 -> 1.76 mm
- net Net-(U2-VBACKUP): track 0.00 -> 1.71 mm

Commit message: mic and speaker
Parts:
- moved J1 218.1 mm to (89.2, 90.0)
- moved C52 205.1 mm to (105.2, 83.2)
- moved J21 205.1 mm to (116.6, 79.0)
- moved J27 198.7 mm to (124.2, 129.2), turned to 90 degrees
- moved J14 198.6 mm to (154.6, 79.6)
- moved J20 192.2 mm to (157.5, 88.4)
- moved Q5 192.2 mm to (160.1, 95.2)
- moved R83 192.2 mm to (157.5, 97.8)
- moved R84 192.2 mm to (160.1, 98.2)
- moved R85 192.2 mm to (156.7, 94.0)
- moved R52 186.8 mm to (144.8, 97.4)
- moved D8 186.8 mm to (148.4, 94.6)
- moved J15 186.8 mm to (145.5, 88.9)
- moved Q2 186.8 mm to (147.6, 97.7)
- moved R53 186.8 mm to (144.6, 94.6)
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Connections:
- net /Peripherials/FAN_PWM renamed /Peripherals/FAN_PWM
- net /Peripherials/INT_RTC renamed /Peripherals/INT_RTC
- net /Peripherials/MATRIX_A renamed /Peripherals/MATRIX_A
- net /Peripherials/MATRIX_B renamed /Peripherals/MATRIX_B
- net /Peripherials/MATRIX_B1 renamed /Peripherals/MATRIX_B1
- net /Peripherials/MATRIX_B2 renamed /Peripherals/MATRIX_B2
- net /Peripherials/MATRIX_C renamed /Peripherals/MATRIX_C
- net /Peripherials/MATRIX_CLK renamed /Peripherals/MATRIX_CLK
- net /Peripherials/MATRIX_D renamed /Peripherals/MATRIX_D
- net /Peripherials/MATRIX_G1 renamed /Peripherals/MATRIX_G1
- net /Peripherials/MATRIX_G2 renamed /Peripherals/MATRIX_G2
- net /Peripherials/MATRIX_LAT renamed /Peripherals/MATRIX_LAT
- net /Peripherials/MATRIX_OE renamed /Peripherals/MATRIX_OE
- net /Peripherials/MATRIX_R1 renamed /Peripherals/MATRIX_R1
- net /Peripherials/MATRIX_R2 renamed /Peripherals/MATRIX_R2
- net /Peripherials/SPI_CS_ESPMini renamed /Peripherals/SPI_CS_ESPMini
- net /Peripherials/SPI_CS_SD_CARD renamed /Peripherals/SPI_CS_SD_CARD
- net /Peripherials/UART_RX_Mini renamed /Peripherals/UART_RX_Mini
- net /Peripherials/UART_TX_Mini renamed /Peripherals/UART_TX_Mini
- net /Peripherials/USB_N_ESP_ESD renamed /Peripherals/USB_N_ESP_ESD
- net /Peripherials/USB_N_ESP_RES renamed /Peripherals/USB_N_ESP_RES
- net /Peripherials/USB_P_ESP_ESD renamed /Peripherals/USB_P_ESP_ESD
- net /Peripherials/USB_P_ESP_RES renamed /Peripherals/USB_P_ESP_RES
- net /Peripherials/VBUS_ESP renamed /Peripherals/VBUS_ESP
- C22 pad 1: /Peripherials/VBUS_STM -> /Peripherals/5V_Buck
- C24 pad 1: /Peripherials/VBUS_STM -> /Peripherals/5V_Buck
- C31 pad 2: +5V -> /Peripherals/5V_Buck
- C56 pad 1: +5V -> /Peripherals/5V_Buck
- D6 pad 1: USB_5V -> +5V
- D7 pad 1: USB_5V -> +5V
- D7 pad 2: /Peripherials/VBUS_STM -> /Peripherals/5V_Buck
- D8 pad 1: 5V -> +5V
- J10 pad 2: 5V -> +5V
- J15 pad 2: 5V -> +5V
- L10 pad 2: +5V -> /Peripherals/5V_Buck
- R63 pad 1: +5V -> /Peripherals/5V_Buck
Routing:
- net /Analog/I2S2_SD: track 1.71 -> 80.1 mm, vias 0 -> 3
- net /Analog/I2S2_CK: track 9.57 -> 85.1 mm, vias 0 -> 2
- net /Analog/RIGHT_SD_MODE: track 0.00 -> 45.7 mm, vias 0 -> 2
- net /Analog/LEFT_SD_MODE: track 0.00 -> 37.1 mm, vias 0 -> 2
- net /Analog/MIC: track 3.10 -> 34.7 mm
- net /ESP32C3/SPI1_CS_ESP: track 2.79 -> 32.6 mm
- net /STM32G4/nRST: track 0.00 -> 15.9 mm, vias 0 -> 2
- net Net-(R18-Pad2): track 0.00 -> 11.0 mm
- net Net-(R17-Pad1): track 0.00 -> 10.7 mm
- net /STM32G4/BOOT0: track 0.00 -> 10.6 mm
- net /ESP32C3/SPI1_MISO: track 65.7 -> 74.6 mm
- net /Peripherals/UART_TX_Mini: track 0.00 -> 7.35 mm
- net 5V: track 9.84 -> 3.59 mm
- net +5V: track 0.00 -> 6.24 mm
- net /Peripherals/UART_RX_Mini: track 0.00 -> 3.91 mm
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
Commit message: done for the day
Parts:
- removed J5: Conn_01x02_Pin, Connector_Molex:Molex_SL_171971-0002_1x02_P2.54mm_Vertical
- moved J19 199.8 mm to (97.2, 92.8)
- moved Q4 199.8 mm to (99.9, 99.6)
- moved R80 199.8 mm to (97.3, 102.3)
- moved R81 199.8 mm to (100.0, 102.5)
- moved R82 199.8 mm to (96.3, 98.3)
- moved C19 195.9 mm to (161.2, 62.9)
- moved R68 195.9 mm to (151.2, 59.5)
- moved R69 195.9 mm to (153.4, 56.9)
- moved R70 195.9 mm to (151.2, 62.5)
- moved R71 195.9 mm to (156.4, 56.9)
- moved U9 195.9 mm to (156.5, 61.2)
- moved H1 186.6 mm to (82.6, 93.0)
- moved C46 166.3 mm to (143.2, 102.0)
- moved R7 166.3 mm to (143.2, 105.0)
- moved R8 166.3 mm to (138.6, 102.0)
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Connections:
- J1 pad 1: /Power/I2C3_SCL -> /Power/I2C3_SDA
- J1 pad 3: /Power/I2C3_SDA -> /Power/I2C3_SCL
- J10 pad 2: +5V -> 5V
- J26 pad 3: +3V3 -> 3V3
- U17 pad 2: +3V3 -> 3V3
- U4 pad 6: +3V3 -> 3V3
Routing:
- net /STM32G4/TV_IR_PWM_1: track 0.00 -> 39.3 mm, vias 0 -> 2
- net /STM32G4/TV_IR_PWM_2: track 0.00 -> 31.4 mm, vias 0 -> 2
- net /STM32G4/I2S3_WS: track 0.00 -> 27.5 mm, vias 0 -> 1
- net /Power/I2C3_SDA: track 0.00 -> 27.4 mm, vias 0 -> 1
- net /STM32G4/I2S3_CK: track 0.00 -> 23.0 mm, vias 0 -> 1
- net /STM32G4/I2S3_SD: track 0.00 -> 21.2 mm, vias 0 -> 1
- net /Power/I2C3_SCL: track 0.00 -> 20.9 mm, vias 0 -> 1
- net /STM32G4/SWDIO: track 0.00 -> 14.5 mm, vias 0 -> 1
- net /STM32G4/SWDCLK: track 0.00 -> 13.5 mm, vias 0 -> 1
- net /STM32G4/BOOT0: track 10.6 -> 20.1 mm
- net 3V3: track 81.7 -> 89.0 mm, vias 28 -> 30
- net /STM32G4/nRST: track 15.9 -> 22.0 mm
- net GND: track 57.5 -> 61.1 mm
- net /Analog/I2S2_SD: track 80.1 -> 77.2 mm
- net /Analog/RIGHT_SD_MODE: track 45.7 -> 46.5 mm

Commit message: Buck routing, general routing / placement, edgecuts and planes
Parts:
- added J5: Conn_01x02_Pin, Connector_Molex:Molex_SL_171971-0002_1x02_P2.54mm_Vertical, F.Cu at (150.4, 94.5)
- C18, J22, R10, R72, R73, R74, R75, R9, U10: moved to B.Cu
- C28, C29: footprint Capacitor_SMD:C_0201_0603Metric_Pad0.64x0.40mm_HandSolder -> Capacitor_SMD:C_0402_1005Metric
- C30, C31, C56, C61, C62, C63, C64, C65, L10, R1, R16, R4, R63, U4: moved to F.Cu
- C78: footprint Package_TO_SOT_SMD:SOT-23-6 -> Capacitor_SMD:C_0603_1608Metric_Pad1.08x0.95mm_HandSolder
- L2: footprint Inductor_SMD:L_0201_0603Metric_Pad0.64x0.40mm_HandSolder -> Inductor_SMD:L_0402_1005Metric
- R86, R88: footprint Resistor_SMD:R_1210_3225Metric_Pad1.30x2.65mm_HandSolder -> Resistor_SMD:R_0805_2012Metric
- moved H2 326.1 mm to (213.4, 149.9)
- moved H3 307.1 mm to (213.4, 94.0)
- moved C22 282.0 mm to (197.1, 161.7), turned to 0 degrees
- moved C24 278.7 mm to (196.3, 159.5), turned to 90 degrees
- moved C23 278.6 mm to (189.1, 161.9), turned to 180 degrees
- moved D7 276.4 mm to (194.3, 158.5), turned to -90 degrees
- moved C25 275.7 mm to (189.9, 159.5), turned to 90 degrees
- moved D6 275.3 mm to (191.9, 158.5), turned to -90 degrees
- moved R72 261.1 mm to (191.1, 127.3)
- moved R73 259.2 mm to (192.8, 127.3), turned to -90 degrees
- moved R74 258.2 mm to (188.3, 125.7), turned to 0 degrees
- moved U10 255.6 mm to (185.7, 129.9), turned to 180 degrees
- moved R75 255.3 mm to (185.3, 125.7), turned to 0 degrees
- moved C18 254.7 mm to (184.0, 133.6), turned to 0 degrees
- moved F1 230.9 mm to (199.1, 144.8), turned to 90 degrees
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Connections:
- J1 pad 1: /Power/I2C3_SDA -> /Power/I2C3_SCL
- J1 pad 3: /Power/I2C3_SCL -> /Power/I2C3_SDA
Routing:
- net /Power/I2C3_SCL: track 20.9 -> 51.3 mm
- net /Power/I2C3_SDA: track 27.4 -> 46.6 mm
- net /Power/VBUS_STM: track 25.0 -> 42.5 mm, vias 0 -> 1
- net /Power/STM32_USB_D_N: track 0.00 -> 14.4 mm
- net /Power/STM32_USB_D_P: track 0.00 -> 13.9 mm
- net Net-(U18-FB): track 0.00 -> 10.1 mm
- net /Analog/I2S2_CK: track 85.3 -> 94.0 mm
- net /Power/3V3_AMPS_1: track 0.00 -> 7.18 mm
- net 3V3: track 89.0 -> 94.2 mm, vias 30 -> 31
- net /STM32G4/USB_VBUS_DETECT: track 0.00 -> 4.67 mm, vias 0 -> 1
- net /STM32G4/ALS_ADC: track 0.00 -> 4.34 mm
- net /Peripherals/USB_P_ESP_ESD: track 1.47 -> 5.71 mm
- net /Peripherals/USB_N_ESP_ESD: track 1.47 -> 5.71 mm
- net /Peripherals/VBUS_ESP: track 9.55 -> 13.8 mm
- net /STM32G4/nRST: track 22.0 -> 17.9 mm
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- added copper zone on B.Cu, net /Power/3V3_AMPS_1
- added copper zone on B.Cu, net 3V3
- added copper zone on In2.Cu, net 3V3
- added copper zone on B.Cu, net GND
- added copper zone on In1.Cu, net GND
- added copper zone on B.Cu, net Net-(U18-SW)
- added copper zone on F.Cu, net Net-(U18-SW)
- added copper zone on B.Cu, net Net-(U18-VIN)
Other:
- board outline added: 142.2 x 72.4 mm

Commit message: working on buck
Parts:
- C28, C29: footprint Capacitor_SMD:C_0402_1005Metric -> Capacitor_SMD:C_0201_0603Metric_Pad0.64x0.40mm_HandSolder
- C30, C61, C62, C63, C64, C65, U4: moved to B.Cu
- C78: footprint Capacitor_SMD:C_0603_1608Metric_Pad1.08x0.95mm_HandSolder -> Package_TO_SOT_SMD:SOT-23-6
- L2: footprint Inductor_SMD:L_0402_1005Metric -> Inductor_SMD:L_0201_0603Metric_Pad0.64x0.40mm_HandSolder
- R86, R88: footprint Resistor_SMD:R_0805_2012Metric -> Resistor_SMD:R_1210_3225Metric_Pad1.30x2.65mm_HandSolder
- moved C23 99.0 mm to (94.2, 133.6), turned to 90 degrees
- moved D6 96.9 mm to (97.6, 136.4), turned to 180 degrees
- moved C25 96.7 mm to (96.6, 134.4), turned to 0 degrees
- moved C30 7.99 mm to (254.8, 121.5), turned to -90 degrees
- moved C64 7.59 mm to (260.3, 121.7), turned to -90 degrees
- moved U4 6.46 mm to (257.6, 122.6), turned to 180 degrees
- moved R16 6.17 mm to (241.8, 120.4)
- moved C61 5.92 mm to (254.3, 117.7), turned to 90 degrees
- moved C63 5.69 mm to (261.1, 117.7), turned to 90 degrees
- moved C31 3.19 mm to (244.5, 122.0)
- moved R4 3.19 mm to (244.5, 125.0)
- moved R63 3.19 mm to (244.6, 123.4)
- moved C65 2.10 mm to (254.9, 124.7), turned to -90 degrees
- moved C62 2.03 mm to (257.7, 117.7), turned to 90 degrees
Connections:
- J1 pad 1: /Power/I2C3_SCL -> /Power/I2C3_SDA
- J1 pad 3: /Power/I2C3_SDA -> /Power/I2C3_SCL
- U12 pad 5: /Power/VBUS_STM -> 3V3
Routing:
- net 20V: track 0.00 -> 22.3 mm, vias 0 -> 6
- net /Power/VBUS_STM: track 42.5 -> 25.0 mm, vias 1 -> 0
- net /STM32G4/INT_TEMP_ALERT: track 0.00 -> 14.7 mm
- net /ESP32C3/SPI1_MISO: track 76.8 -> 88.1 mm, vias 2 -> 4
- net 3V3: track 94.2 -> 101.7 mm, vias 31 -> 39
- net GND: track 60.7 -> 67.1 mm, vias 120 -> 130
- net /Peripherals/VBUS_ESP: track 13.8 -> 19.8 mm
- net Net-(C30-Pad2): track 0.00 -> 5.50 mm
- net Net-(U4-VBST): track 0.00 -> 1.69 mm
- net Net-(U4-MODE): track 0.00 -> 1.37 mm

Commit message: second buck
Parts:
- C30, C61, C62, C63, C64, C65, U4: moved to F.Cu
- L10: moved to B.Cu
- moved L10 24.1 mm to (253.2, 113.8), turned to 0 degrees
- moved C56 23.9 mm to (266.3, 118.8), turned to 180 degrees
- moved C61 19.2 mm to (235.7, 122.5), turned to -90 degrees
- moved C63 19.2 mm to (242.5, 122.5), turned to -90 degrees
- moved C62 19.2 mm to (239.1, 122.5), turned to -90 degrees
- moved R4 18.9 mm to (234.0, 140.8)
- moved C19 15.6 mm to (224.6, 101.9)
- moved R68 15.6 mm to (234.6, 105.3)
- moved R70 15.6 mm to (234.6, 102.3)
- moved R69 15.6 mm to (232.4, 107.9)
- moved R71 15.6 mm to (229.4, 107.9)
- moved U9 15.6 mm to (229.3, 103.6)
- moved C64 15.3 mm to (245.0, 121.7)
- moved U4 9.88 mm to (247.7, 122.6), turned to 0 degrees
- moved C31 8.95 mm to (249.0, 129.7), turned to -90 degrees
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Connections:
- D6 pad 1: +5V -> 5V
- D7 pad 1: +5V -> 5V
- D8 pad 1: +5V -> 5V
- J15 pad 2: +5V -> 5V
- J26 pad 1: +5V -> 5V
Routing:
- net 20V: track 22.3 -> 0.00 mm, vias 6 -> 1
- net 5V: track 3.59 -> 9.84 mm
- net +5V: track 6.24 -> 0.00 mm
- net Net-(C30-Pad2): track 5.50 -> 0.00 mm
- net Net-(U4-PG): track 0.00 -> 3.40 mm
- net Net-(U4-MODE): track 1.37 -> 3.54 mm
- net Net-(U4-FB): track 0.00 -> 1.80 mm
- net GND: vias 130 -> 136
- added copper zone on F.Cu, net +20V
- added copper zone on F.Cu, net /Peripherals/5V_Buck
- added copper zone on F.Cu, net Net-(C30-Pad2)
