File: Sensors.kicad_sch (KiCad schematic)
At the start: 7 parts, among them J1 Conn_01x03_Socket, J4 Conn_01x03_Socket, J5 Conn_01x02_Socket

Commit message: wait
Parts:
- removed J1: Conn_01x03_Socket, Package_SO:HTSSOP-20-1EP_4.4x6.5mm_P0.65mm_EP3.4x6.5mm_ThermalVias, symbol Connector:Conn_01x03_Socket
- removed R? (x2): 10k, Resistor_SMD:R_0603_1608Metric, symbol Device:R
- removed R?: R, Package_SON:WSON-6-1EP_2x2mm_P0.65mm_EP1x1.6mm, symbol Device:R
- removed U?: TMP117xxDRV, Package_SON:WSON-6-1EP_2x2mm_P0.65mm_EP1x1.6mm, symbol Sensor_Temperature:TMP117xxDRV
- added J16: Conn_01x03_Socket, symbol Connector:Conn_01x03_Socket
- added R57, R71, R72: 10k, Resistor_SMD:R_0603_1608Metric, symbol Device:R
- added U11: TMP117xxDRV, Package_SON:WSON-6-1EP_2x2mm_P0.65mm_EP1x1.6mm, symbol Sensor_Temperature:TMP117xxDRV
- J4: footprint (none) -> Connector_PinHeader_2.54mm:PinHeader_1x03_P2.54mm_Vertical
Connections:
- net +3V3: now also J16.1 (Pin_1), R57.1, R71.1, U11.5 (V+)
- net ALS_ADC: now also R72.1
- net EXT_TEMP: now also J4.2 (Pin_2), R71.2
- net GND: now also J16.3 (Pin_3), R72.2, U11.2 (GND), U11.4 (ADD0)
- net I2C3_SCL: now also U11.1 (SCL)
- net I2C3_SDA: now also U11.6 (SDA)
- net PAPIR: now also J16.2 (Pin_2); no longer J4.2 (Pin_2)
- new net INT_TEMP_ALERT: R57.2, U11.3 (ALERT)

Commit message: Major Changes - Schematic Done??
Parts:
- removed J4: Conn_01x03_Socket, Connector_PinHeader_2.54mm:PinHeader_1x03_P2.54mm_Vertical, symbol Connector:Conn_01x03_Socket
- removed R71: 10k, Resistor_SMD:R_0603_1608Metric, symbol Device:R
- added C14, C52: 100n, Capacitor_SMD:C_0603_1608Metric, symbol Device:C
- added J1: Conn_01x04_Pin, Connector_PinHeader_2.54mm:PinHeader_1x04_P2.54mm_Vertical, symbol Connector:Conn_01x04_Pin
- added J21: MIC_I2S_CONNECTOR, Connector_PinSocket_2.54mm:PinSocket_1x06_P2.54mm_Vertical, symbol Connector_Generic:Conn_01x06
- added Q4, Q5: AO3400A, Package_TO_SOT_SMD:SOT-23, symbol Transistor_FET:AO3400A
- added R36: 100k, Resistor_SMD:R_0603_1608Metric, symbol Device:R
- added R80, R83: 10, Resistor_SMD:R_0603_1608Metric, symbol Device:R
- added R81, R84: 10k, Resistor_SMD:R_0603_1608Metric, symbol Device:R
- added R82, R85: 17, Resistor_SMD:R_0603_1608Metric, symbol Device:R
- added TSAL2, TSAL3: LED, LED_SMD:LED_0603_1608Metric, symbol Device:LED
- J2: renamed from J5; footprint (none) -> Connector_PinSocket_2.54mm:PinSocket_1x02_P2.54mm_Vertical
- J3: renamed from J16; footprint (none) -> Connector_PinSocket_2.54mm:PinSocket_1x03_P2.54mm_Vertical
- R3: renamed from R72; value 10k -> 2k2
- renumbered R57 to R2, U11 to U1
Connections:
- net ALS_ADC: now also J2.1 (Pin_1), R3.2; no longer J2.2 (Pin_2), R3.1
- net GND: now also J2.2 (Pin_2), C14.2, C52.2, J1.2 (Pin_2), J21.1 (Pin_1), J21.5 (Pin_5), Q4.2 (S), Q5.2 (S), R36.2, R81.2, R84.2; no longer R3.2
- net I2C3_SCL: now also J1.1 (Pin_1)
- net I2C3_SDA: now also J1.3 (Pin_3)
- net PAPIR: now also R36.1
- net +3V3 renamed 3V3
- net 3V3: now also R3.1, C14.1, C52.1, J1.4 (Pin_4), J21.6 (Pin_6), R82.1, R85.1; no longer J2.1 (Pin_1)
- new net: Q5.1 (G), R83.1, R84.1
- new net: Q5.3 (D), TSAL3.1 (K)
- new net: Q4.1 (G), R80.1, R81.1
- new net: Q4.3 (D), TSAL2.1 (K)
- new net: R82.2, TSAL2.2 (A)
- new net: R85.2, TSAL3.2 (A)
- new net I2S3_CK: J21.4 (Pin_4)
- new net I2S3_SD: J21.3 (Pin_3)
- new net I2S3_WS: J21.2 (Pin_2)
- new net TV_IR_PWM_1: R80.2
- new net TV_IR_PWM_2: R83.2
Other:
- note added: "Digital microphone website : https://www.adafruit.com/product/6049"
- note added: "External Temp: AM2320"
- note added: "IR EMITTER"
- note added: "J1 - 6 Pin Connector to Adafruit ICS-43434 Breakout 1 - SEL → GND 2 - LRCL → MIC_I2S_WS 3 - DOUT → MIC_I2S_SD 4 - BCLK → MIC_I2S_SCK 5 - GND → GND 6 - 3V → +3V3"
- note added: "https://www.adafruit.com/product/3721"
- note removed: "External Temp: DHT22/AM2302"
- note removed: "Info over serial line"
- moved on the sheet: J2, J3, R2, R3, U1

Commit message: Pin swaps
Parts:
- removed TSAL2, TSAL3: LED, LED_SMD:LED_0603_1608Metric, symbol Device:LED
- added J19, J20: Conn_01x02_Socket, Connector_PinSocket_2.54mm:PinSocket_1x02_P2.54mm_Vertical, symbol Connector:Conn_01x02_Socket
Connections:
- net at Q5.3 (D): now also J20.2 (Pin_2)
- net at Q4.3 (D): now also J19.2 (Pin_2)
- net at R82.2: now also J19.1 (Pin_1)
- net at R85.2: now also J20.1 (Pin_1)

Commit message: connectors changed from headers, added SWD conn
Parts:
- J1: footprint Connector_PinHeader_2.54mm:PinHeader_1x04_P2.54mm_Vertical -> Connector_Molex:Molex_SL_171971-0004_1x04_P2.54mm_Vertical
- J19, J2: footprint Connector_PinSocket_2.54mm:PinSocket_1x02_P2.54mm_Vertical -> Connector_Molex:Molex_SL_171971-0002_1x02_P2.54mm_Vertical
- J21: footprint Connector_PinSocket_2.54mm:PinSocket_1x06_P2.54mm_Vertical -> Connector_Molex:Molex_SL_171971-0006_1x06_P2.54mm_Vertical
- J3: footprint Connector_PinSocket_2.54mm:PinSocket_1x03_P2.54mm_Vertical -> Connector_Molex:Molex_SL_171971-0003_1x03_P2.54mm_Vertical
Changed lines of the file:
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@@
 			)
 		)
-		(property "Footprint" "Connector_PinSocket_2.54mm:PinSocket_1x02_P2.54mm_Vertical"
+		(property "Footprint" "Connector_Molex:Molex_SL_171971-0002_1x02_P2.54mm_Vertical"
 			(at 222.25 41.91 0)
 			(hide yes)
@@
 			)
 		)
-		(property "Footprint" "Connector_PinSocket_2.54mm:PinSocket_1x06_P2.54mm_Vertical"
+		(property "Footprint" "Connector_Molex:Molex_SL_171971-0006_1x06_P2.54mm_Vertical"
 			(at 245.11 105.41 0)
 			(hide yes)
@@
 			)
 		)
-		(property "Footprint" "Connector_PinSocket_2.54mm:PinSocket_1x02_P2.54mm_Vertical"
+		(property "Footprint" "Connector_Molex:Molex_SL_171971-0002_1x02_P2.54mm_Vertical"
 			(at 152.4 83.82 0)
 			(hide yes)
@@
 			)
 		)
-		(property "Footprint" "Connector_PinSocket_2.54mm:PinSocket_1x03_P2.54mm_Vertical"
+		(property "Footprint" "Connector_Molex:Molex_SL_171971-0003_1x03_P2.54mm_Vertical"
 			(at 135.89 31.75 0)
 			(hide yes)
@@
 			)
 		)
-		(property "Footprint" "Connector_PinHeader_2.54mm:PinHeader_1x04_P2.54mm_Vertical"
+		(property "Footprint" "Connector_Molex:Molex_SL_171971-0004_1x04_P2.54mm_Vertical"
 			(at 55.88 34.29 0)
 			(hide yes)
