File: Sensors.kicad_sch (KiCad schematic)
At the start: 20 parts, among them J1 Conn_01x04_Pin, J19 Conn_01x02_Socket, J2 Conn_01x02_Socket, J20 Conn_01x02_Socket, J21 MIC_I2S_CONNECTOR, J3 Conn_01x03_Socket, Q4 AO3400A, Q5 AO3400A, U1 TMP117xxDRV

Commit message: Schematic formating
Other:
- note added: "AM2320"
- note added: "EKMB1107111"
- note added: "EXTERNAL TEMP"
- note added: "INTERNAL TEMP SENSOR"
- note added: "LIGHT SENSOR"
- note added: "MICROPHONE"
- note added: "PAPIR SENSOR"
- note added: "TEPT5600"
- note added: "TMP117AIDRVR"
- note removed: "External Temp: AM2320"
- note removed: "Internal Temp: TMP117AIDRVR"
- note removed: "Light Sensor: TEPT5600"
- note removed: "PAPIR Sensor: EKMB1107111"
- moved on the sheet: J2, R3
Changed lines of the file:
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@@
 	(paper "A4")
 	(rectangle
-		(start 104.14 62.23)
-		(end 168.91 106.68)
+		(start 96.52 62.23)
+		(end 161.29 106.68)
 		(stroke
-			(width 0)
-			(type default)
+			(width 0.254)
+			(type solid)
 		)
 		(fill
@@
 	)
 	(rectangle
-		(start 231.14 20.32)
-		(end 276.86 76.2)
+		(start 229.87 21.59)
+		(end 278.13 76.2)
 		(stroke
 			(width 0.254)
-			(type dash)
-			(color 0 0 0 1)
+			(type solid)
 		)
 		(fill
@@
 	)
 	(rectangle
-		(start 17.78 20.32)
-		(end 81.28 53.34)
+		(start 176.53 21.59)
+		(end 224.79 76.2)
 		(stroke
-			(width 0)
-			(type default)
+			(width 0.254)
+			(type solid)
 		)
 		(fill
@@
 	)
 	(rectangle
-		(start 192.278 89.154)
-		(end 262.128 142.24)
+		(start 17.78 20.32)
+		(end 81.28 53.34)
 		(stroke
-			(width 0)
-			(type dash)
+			(width 0.254)
+			(type solid)
 		)
 		(fill
@@
 		(end 168.91 53.34)
 		(stroke
-			(width 0)
-			(type default)
+			(width 0.254)
+			(type solid)
 		)
 		(fill
@@
 		(end 91.44 106.68)
 		(stroke
-			(width 0)
-			(type default)
+			(width 0.254)
+			(type solid)
 		)
 		(fill
@@
 	)
 	(rectangle
-		(start 177.8 20.32)
-		(end 223.52 76.2)
+		(start 191.77 88.9)
+		(end 264.16 143.51)
 		(stroke
 			(width 0.254)
-			(type dash)
-			(color 0 0 0 1)
+			(type solid)
 		)
 		(fill
@@
 		)
 	)
-	(text "Light Sensor: TEPT5600"
+	(text "TEPT5600"
 		(exclude_from_sim no)
-		(at 115.57 60.706 0)
+		(at 155.702 105.41 0)
 		(effects
 			(font
@@
 		)
 	)
-	(text "J1 - 6 Pin Connector to Adafruit ICS-43434 Breakout\n\n1 - SEL  → GND\n2 - LRCL → MIC_I2S_WS\n3 - DOUT → MIC_I2S_SD\n4 - BCLK → MIC_I2S_SCK\n5 - GND  → GND\n6 - 3V   → +3V3"
+	(text "EKMB1107111"
 		(exclude_from_sim no)
-		(at 222.25 133.35 0)
+		(at 160.528 52.07 0)
 		(effects
 			(font
@@
 		)
 	)
-	(text "PAPIR Sensor: EKMB1107111"
+	(text "TMP117AIDRVR"
 		(exclude_from_sim no)
-		(at 110.49 18.796 0)
+		(at 82.55 105.41 0)
 		(effects
 			(font
@@
 		)
 	)
-	(text "IR EMITTER\n"
+	(text "LIGHT SENSOR"
 		(exclude_from_sim no)
-		(at 251.714 18.542 0)
+		(at 110.236 60.452 0)
 		(effects
 			(font
@@
 				(bold yes)
 				(italic yes)
-				(color 0 0 0 1)
 			)
 		)
 	)
-	(text "External Temp: AM2320"
+	(text "MICROPHONE"
 		(exclude_from_sim no)
-		(at 28.956 18.034 0)
+		(at 203.708 87.122 0)
+		(effects
+			(font
+				(size 2.54 2.54)
+				(thickness 0.508)
+				(bold yes)
+				(italic yes)
+				(color 0 0 194 1)
+			)
+		)
+	)
+	(text "J1 - 6 Pin Connector to Adafruit ICS-43434 Breakout\n\n1 - SEL  → GND\n2 - LRCL → MIC_I2S_WS\n3 - DOUT → MIC_I2S_SD\n4 - BCLK → MIC_I2S_SCK\n5 - GND  → GND\n6 - 3V   → +3V3"
+		(exclude_from_sim no)
+		(at 222.25 133.35 0)
 		(effects
 			(font
@@
 		)
 	)
+	(text "IR EMITTER\n"
+		(exclude_from_sim no)
+		(at 240.03 19.812 0)
+		(effects
+			(font
+				(size 2.54 2.54)
+				(thickness 0.508)
+				(bold yes)
+				(italic yes)
+				(color 0 0 194 1)
+			)
+		)
+	)
+	(text "PAPIR SENSOR"
+		(exclude_from_sim no)
+		(at 110.49 18.796 0)
+		(effects
+			(font
+				(size 2.54 2.54)
+				(thickness 0.508)
+				(bold yes)
+				(italic yes)
+			)
+		)
+	)
+	(text "EXTERNAL TEMP"
+		(exclude_from_sim no)
+		(at 32.512 18.288 0)
+		(effects
+			(font
+				(size 2.54 2.54)
+				(thickness 0.508)
+				(bold yes)
+				(italic yes)
+			)
+		)
+	)
 	(text "Digital microphone website : https://www.adafruit.com/product/6049"
 		(exclude_from_sim no)
@@
 		)
 	)
-	(text "Internal Temp: TMP117AIDRVR"
+	(text "INTERNAL TEMP SENSOR"
 		(exclude_from_sim no)
-		(at 32.004 60.96 0)
+		(at 41.148 60.706 0)
 		(effects
 			(font
-				(size 1.27 1.27)
+				(size 2.54 2.54)
+				(thickness 0.508)
+				(bold yes)
+				(italic yes)
 			)
 		)
@@
 	(text "IR EMITTER\n"
 		(exclude_from_sim no)
-		(at 198.374 18.542 0)
+		(at 186.944 20.066 0)
 		(effects
 			(font
@@
 				(bold yes)
 				(italic yes)
-				(color 0 0 0 1)
+				(color 0 0 194 1)
 			)
 		)
@@
 		)
 	)
+	(text "AM2320"
+		(exclude_from_sim no)
+		(at 75.692 51.816 0)
+		(effects
+			(font
+				(size 1.27 1.27)
+			)
+		)
+	)
 	(text ""
 		(exclude_from_sim no)
@@
 	(text_box "I2C Address: 0x48\n\n"
 		(exclude_from_sim no)
-		(at 67.31 100.1917 0)
+		(at 67.31 91.3017 0)
 		(size 20.32 3.9483)
 		(margins 0.9525 0.9525 0.9525 0.9525)
@@
 	)
 	(junction
-		(at 139.7 83.82)
+		(at 132.08 83.82)
 		(diameter 0)
 		(color 0 0 0 0)
@@
 	(wire
 		(pts
-			(xy 139.7 83.82) (xy 147.32 83.82)
+			(xy 132.08 83.82) (xy 139.7 83.82)
 		)
 		(stroke
@@
 	(wire
 		(pts
-			(xy 139.7 86.36) (xy 147.32 86.36)
+			(xy 132.08 86.36) (xy 139.7 86.36)
 		)
 		(stroke
@@
 	(wire
 		(pts
-			(xy 130.81 83.82) (xy 139.7 83.82)
+			(xy 123.19 83.82) (xy 132.08 83.82)
 		)
 		(stroke
@@
 	(wire
 		(pts
-			(xy 139.7 95.25) (xy 139.7 86.36)
+			(xy 132.08 95.25) (xy 132.08 86.36)
 		)
 		(stroke
@@
 	(wire
 		(pts
-			(xy 139.7 68.58) (xy 139.7 71.12)
+			(xy 132.08 68.58) (xy 132.08 71.12)
 		)
 		(stroke
@@
 	(wire
 		(pts
-			(xy 139.7 78.74) (xy 139.7 83.82)
+			(xy 132.08 78.74) (xy 132.08 83.82)
 		)
 		(stroke
@@
 	)
 	(image
-		(at 118.11 96.52)
+		(at 110.49 96.52)
 		(scale 0.656605)
 		(data "iVBORw0KGgoAAAANSUhEUgAAAeAAAAE4CAYAAACDuSDXAAAABHNCSVQICAgIfAhkiAAAIABJREFU"
@@
 	(hierarchical_label "ALS_ADC"
 		(shape input)
-		(at 130.81 83.82 180)
+		(at 123.19 83.82 180)
 		(effects
 			(font
@@
 	(symbol
 		(lib_id "power:GND")
-		(at 139.7 95.25 0)
+		(at 132.08 95.25 0)
 		(unit 1)
 		(body_style 1)
@@
 		(fields_autoplaced yes)
 		(property "Reference" "#PWR09"
-			(at 139.7 101.6 0)
+			(at 132.08 101.6 0)
 			(hide yes)
 			(show_name no)
@@
 		)
 		(property "Value" "GND"
-			(at 139.7 100.33 0)
+			(at 132.08 100.33 0)
 			(show_name no)
 			(do_not_autoplace no)
@@
 		)
 		(property "Footprint" ""
-			(at 139.7 95.25 0)
+			(at 132.08 95.25 0)
 			(hide yes)
 			(show_name no)
@@
 		)
 		(property "Datasheet" ""
-			(at 139.7 95.25 0)
+			(at 132.08 95.25 0)
 			(hide yes)
 			(show_name no)
@@
 		)
 		(property "Description" "Power symbol creates a global label with name \"GND\" , ground"
-			(at 139.7 95.25 0)
+			(at 132.08 95.25 0)
 			(hide yes)
 			(show_name no)
@@
 	(symbol
 		(lib_id "Device:R")
-		(at 139.7 74.93 0)
+		(at 132.08 74.93 0)
 		(unit 1)
 		(body_style 1)
@@
 		(fields_autoplaced yes)
 		(property "Reference" "R3"
-			(at 142.24 73.6599 0)
+			(at 134.62 73.6599 0)
 			(show_name no)
 			(do_not_autoplace no)
@@
 		)
 		(property "Value" "2k2"
-			(at 142.24 76.1999 0)
+			(at 134.62 76.1999 0)
 			(show_name no)
 			(do_not_autoplace no)
@@
 		)
 		(property "Footprint" "Resistor_SMD:R_0603_1608Metric"
-			(at 137.922 74.93 90)
+			(at 130.302 74.93 90)
 			(hide yes)
 			(show_name no)
@@
 		)
 		(property "Datasheet" ""
-			(at 139.7 74.93 0)
+			(at 132.08 74.93 0)
 			(hide yes)
 			(show_name no)
@@
 		)
 		(property "Description" "Resistor"
-			(at 139.7 74.93 0)
+			(at 132.08 74.93 0)
 			(hide yes)
 			(show_name no)
@@
 	(symbol
 		(lib_id "Connector:Conn_01x02_Socket")
-		(at 152.4 83.82 0)
+		(at 144.78 83.82 0)
 		(unit 1)
 		(body_style 1)
@@
 		(dnp no)
 		(property "Reference" "J2"
-			(at 143.51 88.646 0)
+			(at 135.89 88.646 0)
 			(show_name no)
 			(do_not_autoplace no)
@@
 		)
 		(property "Value" "Conn_01x02_Socket"
-			(at 143.51 91.186 0)
+			(at 135.89 91.186 0)
 			(show_name no)
 			(do_not_autoplace no)
@@
 		)
 		(property "Footprint" "Connector_Molex:Molex_SL_171971-0002_1x02_P2.54mm_Vertical"
-			(at 152.4 83.82 0)
+			(at 144.78 83.82 0)
 			(hide yes)
 			(show_name no)
@@
 		)
 		(property "Datasheet" ""
-			(at 152.4 83.82 0)
+			(at 144.78 83.82 0)
 			(hide yes)
 			(show_name no)
@@
 		)
 		(property "Description" "Generic connector, single row, 01x02, script generated"
-			(at 152.4 83.82 0)
+			(at 144.78 83.82 0)
 			(hide yes)
 			(show_name no)
@@
 	(symbol
 		(lib_id "power:+3V3")
-		(at 139.7 68.58 0)
+		(at 132.08 68.58 0)
 		(unit 1)
 		(body_style 1)
@@
 		(dnp no)
 		(property "Reference" "#PWR0142"
-			(at 139.7 72.39 0)
+			(at 132.08 72.39 0)
 			(hide yes)
 			(show_name no)
@@
 		)
 		(property "Value" "3V3"
-			(at 139.7 64.77 0)
+			(at 132.08 64.77 0)
 			(show_name no)
 			(do_not_autoplace no)
@@
 		)
 		(property "Footprint" ""
-			(at 139.7 68.58 0)
+			(at 132.08 68.58 0)
 			(hide yes)
 			(show_name no)
@@
 		)
 		(property "Datasheet" ""
-			(at 139.7 68.58 0)
+			(at 132.08 68.58 0)
 			(hide yes)
 			(show_name no)
@@
 		)
 		(property "Description" "Power symbol creates a global label with name \"+3V3\""
-			(at 139.7 68.58 0)
+			(at 132.08 68.58 0)
 			(hide yes)
 			(show_name no)

Commit message: Schematic tiddy up
Other:
- title: (none) -> Sensors Schematic
Changed lines of the file:
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@@
 	(generator_version "10.0")
 	(paper "A4")
+	(title_block
+		(title "Sensors Schematic")
+		(date "2026-10-17")
+		(rev "0")
+		(comment 1 "Javier Aldana + Issa Haddad + Xander Beal")
+	)
 	(rectangle
 		(start 96.52 62.23)

Commit message: small changes
Parts:
- J20: footprint Connector_PinHeader_2.54mm:PinHeader_1x02_P2.54mm_Vertical -> Connector_Molex:Molex_SL_171971-0002_1x02_P2.54mm_Vertical
Changed lines of the file:
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@@
 			)
 		)
-		(property "Footprint" "Connector_PinHeader_2.54mm:PinHeader_1x02_P2.54mm_Vertical"
+		(property "Footprint" "Connector_Molex:Molex_SL_171971-0002_1x02_P2.54mm_Vertical"
 			(at 275.59 41.91 0)
 			(hide yes)

Commit message: Final PCB from Xander
Connections:
- net I2S3_CK: now also J21.2 (Pin_2); no longer J21.4 (Pin_4)
- net I2S3_WS: now also J21.4 (Pin_4); no longer J21.2 (Pin_2)

Commit message: working on buck
Connections:
- net I2C3_SCL: now also J1.3 (Pin_3); no longer J1.1 (Pin_1)
- net I2C3_SDA: now also J1.1 (Pin_1); no longer J1.3 (Pin_3)
Changed lines of the file:
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@@
 		)
 	)
-	(label "I2C3_SCL"
-		(at 33.02 82.55 0)
+	(label "I2C3_SDA"
+		(at 34.29 36.83 0)
 		(effects
 			(font
@@
 	)
 	(label "I2C3_SCL"
-		(at 34.29 36.83 0)
+		(at 33.02 82.55 0)
 		(effects
 			(font
@@
 		)
 	)
-	(label "I2C3_SDA"
+	(label "I2C3_SCL"
 		(at 34.29 31.75 0)
 		(effects
