File: Wireless.kicad_sch (KiCad schematic)
At the start: 26 parts, among them SW1 SW_Push, SW2 SW_Push, U1 ESP32-C3, Y2 Crystal

Commit message: ESP work
Parts:
- added C39: 10u, symbol Device:C
- C23: value C -> 1u
- C24: value C -> 100n
- L4: value L -> 2n
Connections:
- net +3V3: now also C39.1
- net GND: now also U1.33 (GND), C39.2
- net SPI_SCLK: now reaches U1.12 (MTCK/GPIO6)
- net SPI_MOSI: now reaches U1.13 (MTDO/GPIO7)
- net SPI_CS_ESP: now reaches U1.16 (GPIO10)
- net SPI_MISO: now reaches U1.6 (GPIO2/ADC1_CH2)
- no-connect marks 0 -> 15
Other:
- moved on the sheet: C12, C13, C14, C15, C16, C19, C20, C21, C22, C23, C24, L2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

Commit message: Small Changes
Parts:
- added R8: 10k, Package_DIP:DIP-8_W7.62mm, symbol Device:R
- Y2: value Crystal -> 10MHz
Connections:
- net +3V3: now also R8.1
- net SPI_MISO: now also R8.2

Commit message: Wednesday minor changes
Parts:
- added AE1: Antenna, Package_DFN_QFN:DFN-8-1EP_2x3mm_P0.5mm_EP0.61x2.2mm, symbol Device:Antenna
- added D5, D8: LED, symbol Device:LED
- added J14, J15: Conn_01x04_Pin, Connector:Tag-Connect_TC2030-IDC-NL_2x03_P1.27mm_Vertical, symbol Connector:Conn_01x04_Pin
- added R35: 330R, Package_DIP:DIP-8_W7.62mm, symbol Device:R
- added R37, R38, R39, R40: 0R, Package_DIP:DIP-8_W7.62mm, symbol Device:R
- added R41: 10k, Package_DIP:DIP-8_W7.62mm, symbol Device:R
- added R43: 330, Package_DIP:DIP-8_W7.62mm, symbol Device:R
- U1: value ESP32-C3 -> ESP32-C3FH4
- Y2: value 10MHz -> 40MHz
Connections:
- net +3V3: now also R35.1, R41.1
- net BOOT: now also J15.2 (Pin_2)
- net ESP32_RST: now also J15.1 (Pin_1)
- net GND: now also D5.1 (K), D8.1 (K)
- net RF_ANT: now also AE1.1 (A)
- net SPI_CS_ESP: now also J14.4 (Pin_4), R38.2; no longer U1.16 (GPIO10)
- net SPI_MISO: now also J14.1 (Pin_1), J15.4 (Pin_4), R37.2; no longer U1.6 (GPIO2)
- net SPI_MOSI: now also J14.2 (Pin_2), R40.1; no longer U1.13 (GPIO7)
- net SPI_SCLK: now also J14.3 (Pin_3), R39.1; no longer U1.12 (GPIO6)
- net GPIO8: now reaches U1.14 (GPIO8)
- net GPIO8: now also J15.3 (Pin_3), R41.2
- net TEST_LED: now reaches U1.18 (GPIO11)
- net TEST_LED: now also R43.1
- new net: R40.2, U1.13 (GPIO7)
- new net: R39.2, U1.12 (GPIO6)
- new net: R38.1, U1.16 (GPIO10)
- new net: R37.1, U1.6 (GPIO2)
- new net: D8.2 (A), R43.2
- new net: D5.2 (A), R35.2
- no-connect marks 15 -> 13
Other:
- note added: "BREAKOUTS"
- note added: "TEST LED"
- moved on the sheet: C12, C13, C14, C15, C16, C17, C18, C23, C24, C39, L4, R8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

Commit message: adding esp footprints
Parts:
- removed D5: LED, symbol Device:LED
- removed R35: 330R, Package_DIP:DIP-8_W7.62mm, symbol Device:R
- C12, C13, C14, C15, C16, C17, C18, C23, C24, C30, C31, C39: footprint (none) -> Capacitor_SMD:C_0603_1608Metric
- C19, C20, C21, C22: value C -> DNP; footprint (none) -> Capacitor_SMD:C_0402_1005Metric
- D8: footprint (none) -> LED_SMD:LED_0603_1608Metric
- J14, J15: footprint Connector:Tag-Connect_TC2030-IDC-NL_2x03_P1.27mm_Vertical -> Connector_PinHeader_2.54mm:PinHeader_1x04_P2.54mm_Vertical
- L2: value L -> DNP; footprint Relay_THT:Relay_DPDT_Finder_30.22 -> Inductor_SMD:L_0402_1005Metric
- L3: footprint Relay_THT:Relay_DPDT_Finder_30.22 -> Inductor_SMD:L_0402_1005Metric
- L4: footprint Relay_THT:Relay_DPDT_Finder_30.22 -> Inductor_SMD:L_0603_1608Metric
- R18, R37, R38, R39, R40, R41, R43, R6, R7, R8, R9: footprint Package_DIP:DIP-8_W7.62mm -> Resistor_SMD:R_0603_1608Metric
- SW1, SW2: footprint Package_DIP:DIP-8_W7.62mm -> Button_Switch_THT:SW_PUSH_6mm

Commit message: Major Changes - Schematic Done??
Parts:
- removed C30, C31: 1u, Capacitor_SMD:C_0603_1608Metric, symbol Device:C
- removed R18, R6, R7, R9: 10k, Resistor_SMD:R_0603_1608Metric, symbol Device:R
- removed SW1, SW2: SW_Push, Button_Switch_THT:SW_PUSH_6mm, symbol Switch:SW_Push
- added C45: 100n, Capacitor_SMD:C_0603_1608Metric, symbol Device:C
- added R76: 1k, Resistor_SMD:R_0603_1608Metric, symbol Device:R
- added R78, R79: 10k, Resistor_SMD:R_0603_1608Metric, symbol Device:R
- added SW6, SW7: SW_Push, Button_Switch_THT:SW_PUSH_6mm, symbol Switch:SW_Push
- AE1: footprint Package_DFN_QFN:DFN-8-1EP_2x3mm_P0.5mm_EP0.61x2.2mm -> RF_Antenna:Texas_SWRA117D_2.4GHz_Left
- C26: renamed from C17; value C -> 22p
- C27: renamed from C18; value C -> 22p
- L2: renamed from L3; value L -> DNP
- L4: footprint Inductor_SMD:L_0603_1608Metric -> Inductor_SMD:L_0402_1005Metric
- Y2: footprint Package_QFP:LQFP-64_10x10mm_P0.5mm -> Crystal:Crystal_SMD_ECS_CSM3X-2Pin_7.6x4.1mm
- renumbered C22 to C28, C19 to C29, C20 to C30, C21 to C31, C13 to C32, C23 to C33, C14 to C34, C15 to C35, C24 to C36, C16 to C37, C39 to C38, C12 to C39, D8 to D9, J14 to J16, J15 to J17, L2 to L3, R43 to R54, R39 to R55, R40 to R56, R37 to R57, R38 to R58, R41 to R59, R8 to R60, U1 to U14
Connections:
- net BOOT: now also R79.2, SW7.1
- net ESP32_RST: now also C45.1, R76.1
- net GND: now also C45.2, SW6.2, SW7.2
- net +3V3 renamed 3V3
- net 3V3: now also R78.1, R79.1
- net SPI_MISO renamed SPI1_MISO
- net SPI_MOSI renamed SPI1_MOSI
- net SPI_SCLK renamed SPI1_SCLK
- new net: R76.2, R78.2, SW6.1
Other:
- moved on the sheet: C26, C27, D9, R54

Commit message: PCB Work
Parts:
- L4: footprint Inductor_SMD:L_0402_1005Metric -> Inductor_SMD:L_0603_1608Metric_Pad1.05x0.95mm_HandSolder
Connections:
- net BOOT: now also J17.3 (Pin_3); no longer J17.2 (Pin_2)
- net GPIO8: now also J17.2 (Pin_2); no longer J17.3 (Pin_3)
Changed lines of the file:
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@@
 	(wire
 		(pts
-			(xy 80.01 52.07) (xy 95.25 52.07)
-		)
-		(stroke
-			(width 0)
-			(type default)
-		)
-	)
-	(wire
-		(pts
 			(xy 194.31 25.4) (xy 194.31 26.67)
 		)
@@
 	(wire
 		(pts
+			(xy 80.01 52.07) (xy 95.25 52.07)
+		)
+		(stroke
+			(width 0)
+			(type default)
+		)
+	)
+	(wire
+		(pts
 			(xy 39.37 45.72) (xy 39.37 48.26)
 		)
@@
 	(wire
 		(pts
+			(xy 80.01 49.53) (xy 95.25 49.53)
+		)
+		(stroke
+			(width 0)
+			(type default)
+		)
+	)
+	(wire
+		(pts
 			(xy 182.88 26.67) (xy 182.88 27.94)
 		)
@@
 	(wire
 		(pts
-			(xy 80.01 49.53) (xy 95.25 49.53)
-		)
-		(stroke
-			(width 0)
-			(type default)
-		)
-	)
-	(wire
-		(pts
 			(xy 256.54 110.49) (xy 256.54 113.03)
 		)
@@
 	)
 	(label "BOOT"
-		(at 80.01 52.07 0)
+		(at 80.01 49.53 0)
 		(effects
 			(font
@@
 	)
 	(label "GPIO8"
-		(at 80.01 49.53 0)
+		(at 80.01 52.07 0)
 		(effects
 			(font
@@
 			)
 		)
-		(property "Footprint" "Inductor_SMD:L_0402_1005Metric"
+		(property "Footprint" "Inductor_SMD:L_0603_1608Metric_Pad1.05x0.95mm_HandSolder"
 			(at 175.26 26.67 0)
 			(hide yes)

Commit message: Minor PCB Changes
Parts:
- removed AE1: Antenna, RF_Antenna:Texas_SWRA117D_2.4GHz_Left, symbol Device:Antenna
- added AE1: Antenna_Shield, RF_Antenna:Texas_SWRA117D_2.4GHz_Left, symbol Device:Antenna_Shield
- added J11: Conn_01x02_Pin, Connector_PinHeader_2.54mm:PinHeader_1x02_P2.54mm_Vertical, symbol Connector:Conn_01x02_Pin
Connections:
- net GND: now also AE1.2 (Shield)
- net RF_ANT: now also AE1.1 (A)
- net UART_RX: now reaches U14.27 (GPIO20)
- net UART_RX: now also J11.2 (Pin_2)
- net UART_TX: now reaches U14.28 (GPIO21)
- net UART_TX: now also J11.1 (Pin_1)
- no-connect marks 13 -> 11

Commit message: Schematic tiddy up
Connections:
- net VDD3P3: now reaches C33.1, L4.1, U14.2 (VDD3P3), U14.3 (VDD3P3)
Other:
- note added: "ANTENNA"
- note added: "BOOT BUTTON"
- note added: "ESP32"
- note added: "PWR CAPS"
- note added: "RESET BUTTON"
- note removed: "RESET AND BOOT BUTTONS"
- title: (none) -> ESP32 Schematic
- moved on the sheet: AE1, C26, C27, C28, C29, C30, C31, C32, C33, C34, C35, C36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
