File: Wireless.kicad_sch (KiCad schematic)
At the start: 37 parts, among them J11 Conn_01x02_Pin, J16 Conn_01x04_Pin, J17 Conn_01x04_Pin, SW6 SW_Push, SW7 SW_Push, U14 ESP32-C3FH4, Y2 40MHz

Commit message: small changes
Other:
- moved on the sheet: AE1, C26, C27, C28, C29, C30, C31, C32, C33, C34, C35, C36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

Commit message: Final PCB from Xander
Other:
- moved on the sheet: C33
Changed lines of the file:
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@@
 	)
 	(junction
-		(at 25.4 140.97)
+		(at 22.86 140.97)
 		(diameter 0)
 		(color 0 0 0 0)
@@
 	)
 	(junction
+		(at 27.94 140.97)
+		(diameter 0)
+		(color 0 0 0 0)
+	)
+	(junction
 		(at 69.85 38.1)
 		(diameter 0)
@@
 	(wire
 		(pts
+			(xy 27.94 140.97) (xy 29.21 140.97)
+		)
+		(stroke
+			(width 0)
+			(type default)
+		)
+	)
+	(wire
+		(pts
 			(xy 36.83 102.87) (xy 31.75 102.87)
 		)
@@
 	(wire
 		(pts
-			(xy 34.29 43.18) (xy 34.29 35.56)
+			(xy 35.56 43.18) (xy 35.56 35.56)
 		)
 		(stroke
@@
 	(wire
 		(pts
-			(xy 25.4 140.97) (xy 29.21 140.97)
+			(xy 22.86 140.97) (xy 27.94 140.97)
 		)
 		(stroke
@@
 	(wire
 		(pts
-			(xy 25.4 139.7) (xy 25.4 140.97)
+			(xy 22.86 139.7) (xy 22.86 140.97)
 		)
 		(stroke
@@
 	(wire
 		(pts
-			(xy 166.37 34.29) (xy 166.37 41.91)
+			(xy 166.37 35.56) (xy 166.37 41.91)
 		)
 		(stroke
@@
 	(wire
 		(pts
-			(xy 25.4 140.97) (xy 25.4 142.24)
+			(xy 22.86 140.97) (xy 22.86 142.24)
 		)
 		(stroke
@@
 	(wire
 		(pts
-			(xy 25.4 151.13) (xy 52.07 151.13)
+			(xy 22.86 151.13) (xy 52.07 151.13)
 		)
 		(stroke
@@
 	(wire
 		(pts
-			(xy 25.4 149.86) (xy 25.4 151.13)
+			(xy 22.86 149.86) (xy 22.86 151.13)
 		)
 		(stroke
@@
 	(wire
 		(pts
-			(xy 34.29 35.56) (xy 31.75 35.56)
+			(xy 35.56 35.56) (xy 31.75 35.56)
 		)
 		(stroke
@@
 	(symbol
 		(lib_id "power:+3V3")
-		(at 25.4 139.7 0)
+		(at 22.86 139.7 0)
 		(unit 1)
 		(body_style 1)
@@
 		(dnp no)
 		(property "Reference" "#PWR0161"
-			(at 25.4 143.51 0)
+			(at 22.86 143.51 0)
 			(hide yes)
 			(show_name no)
@@
 		)
 		(property "Value" "VDD3P3"
-			(at 25.4 136.144 0)
+			(at 22.86 136.144 0)
 			(show_name no)
 			(do_not_autoplace no)
@@
 		)
 		(property "Footprint" ""
-			(at 25.4 139.7 0)
+			(at 22.86 139.7 0)
 			(hide yes)
 			(show_name no)
@@
 		)
 		(property "Datasheet" ""
-			(at 25.4 139.7 0)
+			(at 22.86 139.7 0)
 			(hide yes)
 			(show_name no)
@@
 		)
 		(property "Description" "Power symbol creates a global label with name \"+3V3\""
-			(at 25.4 139.7 0)
+			(at 22.86 139.7 0)
 			(hide yes)
 			(show_name no)
@@
 	)
 	(symbol
+		(lib_id "power:PWR_FLAG")
+		(at 27.94 140.97 0)
+		(unit 1)
+		(body_style 1)
+		(exclude_from_sim no)
+		(in_bom yes)
+		(on_board yes)
+		(in_pos_files yes)
+		(dnp no)
+		(property "Reference" "#FLG06"
+			(at 27.94 139.065 0)
+			(hide yes)
+			(show_name no)
+			(do_not_autoplace no)
+			(effects
+				(font
+					(size 1.27 1.27)
+				)
+			)
+		)
+		(property "Value" "PWR_FLAG"
+			(at 28.194 137.922 0)
+			(show_name no)
+			(do_not_autoplace no)
+			(effects
+				(font
+					(size 1.27 1.27)
+				)
+			)
+		)
+		(property "Footprint" ""
+			(at 27.94 140.97 0)
+			(hide yes)
+			(show_name no)
+			(do_not_autoplace no)
+			(effects
+				(font
+					(size 1.27 1.27)
+				)
+			)
+		)
+		(property "Datasheet" ""
+			(at 27.94 140.97 0)
+			(hide yes)
+			(show_name no)
+			(do_not_autoplace no)
+			(effects
+				(font
+					(size 1.27 1.27)
+				)
+			)
+		)
+		(property "Description" "Special symbol for telling ERC where power comes from"
+			(at 27.94 140.97 0)
+			(hide yes)
+			(show_name no)
+			(do_not_autoplace no)
+			(effects
+				(font
+					(size 1.27 1.27)
+				)
+			)
+		)
+		(pin "1"
+		)
+		(instances
+			(project "SeniorDesign_PCB"
+				(path "/88e1ced0-9576-4565-ab29-f74bf51ccbda/8dbcbcde-a963-4a54-aef5-5a4212c7899c"
+					(reference "#FLG06")
+					(unit 1)
+				)
+			)
+		)
+	)
+	(symbol
 		(lib_id "power:+3V3")
 		(at 140.97 132.08 0)
@@
 	)
 	(symbol
+		(lib_id "power:GND")
+		(at 35.56 43.18 0)
+		(unit 1)
+		(body_style 1)
+		(exclude_from_sim no)
+		(in_bom yes)
+		(on_board yes)
+		(in_pos_files yes)
+		(dnp no)
+		(property "Reference" "#PWR0108"
+			(at 35.56 49.53 0)
+			(hide yes)
+			(show_name no)
+			(do_not_autoplace no)
+			(effects
+				(font
+					(size 1.27 1.27)
+				)
+			)
+		)
+		(property "Value" "GND"
+			(at 35.56 46.99 0)
+			(show_name no)
+			(do_not_autoplace no)
+			(effects
+				(font
+					(size 1.27 1.27)
+				)
+			)
+		)
+		(property "Footprint" ""
+			(at 35.56 43.18 0)
+			(hide yes)
+			(show_name no)
+			(do_not_autoplace no)
+			(effects
+				(font
+					(size 1.27 1.27)
+				)
+			)
+		)
+		(property "Datasheet" ""
+			(at 35.56 43.18 0)
+			(hide yes)
+			(show_name no)
+			(do_not_autoplace no)
+			(effects
+				(font
+					(size 1.27 1.27)
+				)
+			)
+		)
+		(property "Description" "Power symbol creates a global label with name \"GND\" , ground"
+			(at 35.56 43.18 0)
+			(hide yes)
+			(show_name no)
+			(do_not_autoplace no)
+			(effects
+				(font
+					(size 1.27 1.27)
+				)
+			)
+		)
+		(pin "1"
+		)
+		(instances
+			(project "SeniorDesign_PCB"
+				(path "/88e1ced0-9576-4565-ab29-f74bf51ccbda/8dbcbcde-a963-4a54-aef5-5a4212c7899c"
+					(reference "#PWR0108")
+					(unit 1)
+				)
+			)
+		)
+	)
+	(symbol
 		(lib_id "Device:R")
 		(at 215.9 66.04 0)
@@
 	(symbol
 		(lib_id "power:GND")
-		(at 34.29 43.18 0)
-		(unit 1)
-		(body_style 1)
-		(exclude_from_sim no)
-		(in_bom yes)
-		(on_board yes)
-		(in_pos_files yes)
-		(dnp no)
-		(property "Reference" "#PWR0108"
-			(at 34.29 49.53 0)
-			(hide yes)
-			(show_name no)
-			(do_not_autoplace no)
-			(effects
-				(font
-					(size 1.27 1.27)
-				)
-			)
-		)
-		(property "Value" "GND"
-			(at 34.29 46.99 0)
-			(show_name no)
-			(do_not_autoplace no)
-			(effects
-				(font
-					(size 1.27 1.27)
-				)
-			)
-		)
-		(property "Footprint" ""
-			(at 34.29 43.18 0)
-			(hide yes)
-			(show_name no)
-			(do_not_autoplace no)
-			(effects
-				(font
-					(size 1.27 1.27)
-				)
-			)
-		)
-		(property "Datasheet" ""
-			(at 34.29 43.18 0)
-			(hide yes)
-			(show_name no)
-			(do_not_autoplace no)
-			(effects
-				(font
-					(size 1.27 1.27)
-				)
-			)
-		)
-		(property "Description" "Power symbol creates a global label with name \"GND\" , ground"
-			(at 34.29 43.18 0)
-			(hide yes)
-			(show_name no)
-			(do_not_autoplace no)
-			(effects
-				(font
-					(size 1.27 1.27)
-				)
-			)
-		)
-		(pin "1"
-		)
-		(instances
-			(project "SeniorDesign_PCB"
-				(path "/88e1ced0-9576-4565-ab29-f74bf51ccbda/8dbcbcde-a963-4a54-aef5-5a4212c7899c"
-					(reference "#PWR0108")
-					(unit 1)
-				)
-			)
-		)
-	)
-	(symbol
-		(lib_id "power:GND")
 		(at 86.36 157.48 0)
 		(unit 1)
@@
 	(symbol
 		(lib_id "power:+3V3")
-		(at 166.37 34.29 0)
+		(at 166.37 35.56 0)
 		(unit 1)
 		(body_style 1)
@@
 		(dnp no)
 		(property "Reference" "#PWR0160"
-			(at 166.37 38.1 0)
+			(at 166.37 39.37 0)
 			(hide yes)
 			(show_name no)
@@
 		)
 		(property "Value" "VDD3P3"
-			(at 166.37 30.734 0)
+			(at 166.37 32.004 0)
 			(show_name no)
 			(do_not_autoplace no)
@@
 		)
 		(property "Footprint" ""
-			(at 166.37 34.29 0)
+			(at 166.37 35.56 0)
 			(hide yes)
 			(show_name no)
@@
 		)
 		(property "Datasheet" ""
-			(at 166.37 34.29 0)
+			(at 166.37 35.56 0)
 			(hide yes)
 			(show_name no)
@@
 		)
 		(property "Description" "Power symbol creates a global label with name \"+3V3\""
-			(at 166.37 34.29 0)
+			(at 166.37 35.56 0)
 			(hide yes)
 			(show_name no)
@@
 	(symbol
 		(lib_id "Device:C")
-		(at 25.4 146.05 0)
+		(at 22.86 146.05 0)
 		(unit 1)
 		(body_style 1)
@@
 		(dnp no)
 		(property "Reference" "C33"
-			(at 25.654 143.764 0)
+			(at 23.114 143.764 0)
 			(show_name no)
 			(do_not_autoplace no)
@@
 		)
 		(property "Value" "1u"
-			(at 25.654 148.082 0)
+			(at 23.114 148.082 0)
 			(show_name no)
 			(do_not_autoplace no)
@@
 		)
 		(property "Footprint" "Capacitor_SMD:C_0603_1608Metric"
-			(at 26.3652 149.86 0)
+			(at 23.8252 149.86 0)
 			(hide yes)
 			(show_name no)
@@
 		)
 		(property "Datasheet" ""
-			(at 25.4 146.05 0)
+			(at 22.86 146.05 0)
 			(hide yes)
 			(show_name no)
@@
 		)
 		(property "Description" "Unpolarized capacitor"
-			(at 25.4 146.05 0)
+			(at 22.86 146.05 0)
 			(hide yes)
 			(show_name no)

Commit message: wireless work
Parts:
- removed C30, C31: DNP, Capacitor_SMD:C_0402_1005Metric, symbol Device:C
- removed L3: DNP, Inductor_SMD:L_0402_1005Metric, symbol Device:L
- C28, C29: footprint Capacitor_SMD:C_0402_1005Metric -> Capacitor_SMD:C_0201_0603Metric_Pad0.64x0.40mm_HandSolder
- L2: footprint Inductor_SMD:L_0402_1005Metric -> Inductor_SMD:L_0201_0603Metric_Pad0.64x0.40mm_HandSolder
Connections:
- net L_to_L is gone; now on net LNA_IN: C29.1, L2.2
