File: Peripherials.kicad_sch (KiCad schematic)
At the start: 25 parts, among them J13 USB_C_Receptacle_USB2.0_14P, J14 IDC_Cable_02x08, J15 Conn_01x02_Pin, J18 Micro_SD_Card, Q2 NMOS, U13 USBLC6-2P6, U2 RV-3028-C7

Commit message: fixing xander's push
Parts:
- added H1, H2, H3, H4: MountingHole, MountingHole:MountingHole_3.2mm_M3, symbol Mechanical:MountingHole
- added J26, J9: Conn_01x08_Socket, Connector_PinHeader_2.54mm:PinHeader_1x08_P2.54mm_Vertical, symbol Connector:Conn_01x08_Socket
- added J27: Conn_01x02_Socket, Connector_PinHeader_2.54mm:PinHeader_1x02_P2.54mm_Vertical, symbol Connector:Conn_01x02_Socket
Connections:
- net GND: now also J26.2 (Pin_2)
- net SPI1_MISO: now also J9.1 (Pin_1)
- net SPI1_MOSI: now also J9.2 (Pin_2)
- net SPI1_SCLK: now also J9.3 (Pin_3)
- new net +3V3: J26.3 (Pin_3)
- new net +5V: J26.1 (Pin_1)
- new net SPI_CS_ESPMini: J9.6 (Pin_6)
- new net UART_RX_Mini: J27.2 (Pin_2), J9.8 (Pin_8)
- new net UART_TX_Mini: J27.1 (Pin_1), J9.7 (Pin_7)
- no-connect marks 3 -> 10
Other:
- note added: "ESP32 Mini Header"
- note added: "Mounting Holes"
- note added: "UART breakout"

Commit message: saving progress
Connections:
- net +3V3 is gone; now on net 3V3: J26.3 (Pin_3)
- net 5V is gone; now on net +5V: D8.1 (K), J15.2 (Pin_2)
- net USB_5V is gone; now on net +5V: D6.1 (K), D7.1 (K)
- net VBUS_STM renamed 5V_Buck
Changed lines of the file:
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@@
 	(wire
 		(pts
-			(xy 130.81 29.21) (xy 146.05 29.21)
+			(xy 139.7 29.21) (xy 146.05 29.21)
 		)
 		(stroke
@@
 		)
 	)
-	(label "VBUS_STM"
-		(at 130.81 29.21 0)
-		(effects
-			(font
-				(size 1.27 1.27)
-			)
-			(justify left bottom)
-		)
-	)
 	(label "UART_RX_Mini"
 		(at 240.03 105.41 180)
@@
 		)
 	)
+	(hierarchical_label "5V_Buck"
+		(shape input)
+		(at 139.7 29.21 180)
+		(effects
+			(font
+				(size 1.27 1.27)
+			)
+			(justify right)
+		)
+	)
 	(hierarchical_label "ESP32_USB_D_N"
 		(shape input)
@@
 			)
 		)
-		(property "Value" "USB_5V"
+		(property "Value" "+5V"
 			(at 172.72 22.86 0)
 			(show_name no)
@@
 			)
 		)
-		(property "Value" "+3V3"
-			(at 72.39 161.29 0)
+		(property "Value" "3V3"
+			(at 74.93 165.0999 0)
 			(show_name no)
 			(do_not_autoplace no)
@@
 					(size 1.27 1.27)
 				)
+				(justify left)
 			)
 		)
@@
 			)
 		)
-		(property "Value" "5V"
+		(property "Value" "+5V"
 			(at 222.25 22.86 0)
 			(show_name no)

Commit message: second buck
Connections:
- net +5V renamed 5V
Changed lines of the file:
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@@
 			)
 		)
-		(property "Value" "+5V"
+		(property "Value" "5V"
 			(at 172.72 22.86 0)
 			(show_name no)
@@
 			)
 		)
-		(property "Value" "+5V"
-			(at 77.47 161.29 0)
+		(property "Value" "5V"
+			(at 80.01 165.0999 0)
 			(show_name no)
 			(do_not_autoplace no)
@@
 					(size 1.27 1.27)
 				)
+				(justify left)
 			)
 		)
@@
 			)
 		)
-		(property "Value" "+5V"
+		(property "Value" "5V"
 			(at 222.25 22.86 0)
 			(show_name no)

Commit message: Matrix routing plus pwr
Connections:
- net 5V_Buck: no longer names the net of C22.1, C24.1, D7.2 (A)
Changed lines of the file:
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@@
-		)
-	)
-	(hierarchical_label "5V_Buck"
-		(shape input)
-		(at 139.7 29.21 180)
-		(effects
-			(font
-				(size 1.27 1.27)
-			)
-			(justify right)
 		)
 	)

Commit message: 5V fix
Connections:
- net 5V_Buck: now reaches C22.1, C24.1, D7.2 (A)
Changed lines of the file:
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@@
+		)
+	)
+	(hierarchical_label "5V_Buck"
+		(shape input)
+		(at 139.7 29.21 180)
+		(effects
+			(font
+				(size 1.27 1.27)
+			)
+			(justify right)
 		)
 	)

Commit message: minor Schematic fixes
Parts:
- added Q11: NMOS, Package_TO_SOT_SMD:TSOT-23, symbol Simulation_SPICE:NMOS
- added R33: 10R, Resistor_SMD:R_0603_1608Metric, symbol Device:R
- added R39: 10k, Resistor_SMD:R_0603_1608Metric, symbol Device:R
Connections:
- net GND: now also Q11.3 (S), R39.2; no longer J14.13 (Pin_13), J14.15 (Pin_15), J14.9 (Pin_9)
- net MATRIX_A: now also J14.9 (Pin_5); no longer J14.5 (Pin_5)
- net MATRIX_B: now also J14.10 (Pin_12); no longer J14.12 (Pin_12)
- net MATRIX_B1: now also J14.3 (Pin_2); no longer J14.2 (Pin_2)
- net MATRIX_B2: now also J14.7 (Pin_4); no longer J14.4 (Pin_4)
- net MATRIX_C: now also J14.11 (Pin_6); no longer J14.6 (Pin_6)
- net MATRIX_CLK: now also J14.13 (Pin_7); no longer J14.7 (Pin_7)
- net MATRIX_D: now also J14.12 (Pin_11); no longer J14.11 (Pin_11)
- net MATRIX_G1: now also J14.2 (Pin_16); no longer J14.16 (Pin_16)
- net MATRIX_G2: now also J14.6 (Pin_14); no longer J14.14 (Pin_14)
- net MATRIX_LAT: now also J14.14 (Pin_10); no longer J14.10 (Pin_10)
- net MATRIX_OE: now also J14.15 (Pin_8); no longer J14.8 (Pin_8)
- net MATRIX_R2: now also J14.5 (Pin_3); no longer J14.3 (Pin_3)
- new net: J14.16 (Pin_9), J14.4 (Pin_15), J14.8 (Pin_13), Q11.1 (D)
- new net: Q11.2 (G), R33.2, R39.1
- new net MATRIX_PWR_EN: R33.1
